File: TACTILE_20UFQFPN_SPI_v2.0/TACTILE_STM32L011F4_SPI_v2.0.kicad_sch (KiCad schematic)
At the start: 24 parts, among them U2 DRV5057A1QDBZR, U3 DRV5057A1QDBZR, U4 DRV5057A1QDBZR, U5 DRV5057A1QDBZR

Commit message: update tactile pcb v2.0
Parts:
- U2, U3, U4, U5: value DRV5057A1QDBZR -> DRV5056A4
