File: TACTILE_28UFQFPN_SPI_v2.0/TACTILE_28UFQFPN_SPI_v2.0.kicad_pcb (KiCad board)
At the start: 2 copper layers, 20 x 32 mm, 20 parts, among them J1 59453-061110ECHLF, J2 59453-061110ECHLF, U1 STM32G071G8U6N, U2 DRV5057A1QDBZR, U3 DRV5057A1QDBZR, U4 DRV5057A1QDBZR, U5 DRV5057A1QDBZR

Commit message: update tactile pcb v2.0
Parts:
- U2, U3, U4, U5: value DRV5057A1QDBZR -> DRV5056A4
Changed lines of the file:
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@@
       (effects (font (size 1.1684 1.1684) (thickness 0.1016)) (justify left bottom))
     )
-    (fp_text value "DRV5057A1QDBZR" (at -1.905 3.175 90) (layer "F.Fab")
+    (fp_text value "DRV5056A4" (at -1.905 3.175 90) (layer "F.Fab")
       (effects (font (size 1.1684 1.1684) (thickness 0.1016)) (justify left bottom))
     )
@@
       (effects (font (size 1.1684 1.1684) (thickness 0.1016)) (justify left bottom))
     )
-    (fp_text value "DRV5057A1QDBZR" (at -1.905 3.175 -90) (layer "F.Fab")
+    (fp_text value "DRV5056A4" (at -1.905 3.175 -90) (layer "F.Fab")
       (effects (font (size 1.1684 1.1684) (thickness 0.1016)) (justify left bottom))
     )
@@
       (effects (font (size 1.1684 1.1684) (thickness 0.1016)) (justify left bottom))
     )
-    (fp_text value "DRV5057A1QDBZR" (at -1.905 3.175 -90) (layer "F.Fab")
+    (fp_text value "DRV5056A4" (at -1.905 3.175 -90) (layer "F.Fab")
       (effects (font (size 1.1684 1.1684) (thickness 0.1016)) (justify left bottom))
     )
@@
       (effects (font (size 1.1684 1.1684) (thickness 0.1016)) (justify left bottom))
     )
-    (fp_text value "DRV5057A1QDBZR" (at -1.905 3.175 90) (layer "F.Fab")
-      (effects (font (size 1.1684 1.1684) (thickness 0.1016)) (justify left bottom))
-    )
+    (fp_text value "DRV5056A4" (at -1.905 3.175 90) (layer "F.Fab")
+      (effects (font (size 1.1684 1.1684) (thickness 0.1016)) (justify left bottom))
+    )
