File: TACTILE_28UFQFPN_SPI_v2.0/TACTILE_28UFQFPN_SPI_v2.0.kicad_sch (KiCad schematic)
At the start: 20 parts, among them J1 59453-061110ECHLF, J2 59453-061110ECHLF, U1 STM32G071G8U6N, U2 DRV5057A1QDBZR, U3 DRV5057A1QDBZR, U4 DRV5057A1QDBZR, U5 DRV5057A1QDBZR

Commit message: update tactile pcb v2.0
Parts:
- C3, C4, C5, C6: value C-EUC0402 -> 100nF
- U2, U3, U4, U5: value DRV5057A1QDBZR -> DRV5056A4
Changed lines of the file:
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@@
       (effects (font (size 1.778 1.5113)) (justify left bottom))
     )
-    (property "Value" "C-EUC0402" (id 1) (at 141.224 113.919 0)
+    (property "Value" "100nF" (id 1) (at 141.224 113.919 0)
       (effects (font (size 1.778 1.5113)) (justify left bottom))
     )
@@
       (effects (font (size 1.778 1.5113)) (justify left bottom))
     )
-    (property "Value" "C-EUC0402" (id 1) (at 141.224 141.859 0)
+    (property "Value" "100nF" (id 1) (at 141.224 141.859 0)
       (effects (font (size 1.778 1.5113)) (justify left bottom))
     )
@@
       (effects (font (size 1.778 1.5113)) (justify left bottom))
     )
-    (property "Value" "C-EUC0402" (id 1) (at 141.224 167.259 0)
+    (property "Value" "100nF" (id 1) (at 141.224 167.259 0)
       (effects (font (size 1.778 1.5113)) (justify left bottom))
     )
@@
       (effects (font (size 1.778 1.5113)) (justify left bottom))
     )
-    (property "Value" "C-EUC0402" (id 1) (at 141.224 192.659 0)
+    (property "Value" "100nF" (id 1) (at 141.224 192.659 0)
       (effects (font (size 1.778 1.5113)) (justify left bottom))
     )
@@
       (effects (font (size 1.778 1.5113)) (justify left bottom))
     )
-    (property "Value" "DRV5057A1QDBZR" (id 1) (at 100.33 119.38 0)
+    (property "Value" "DRV5056A4" (id 1) (at 100.33 119.38 0)
       (effects (font (size 1.778 1.5113)) (justify left bottom))
     )
@@
       (effects (font (size 1.778 1.5113)) (justify left bottom))
     )
-    (property "Value" "DRV5057A1QDBZR" (id 1) (at 100.33 147.32 0)
+    (property "Value" "DRV5056A4" (id 1) (at 100.33 147.32 0)
       (effects (font (size 1.778 1.5113)) (justify left bottom))
     )
@@
       (effects (font (size 1.778 1.5113)) (justify left bottom))
     )
-    (property "Value" "DRV5057A1QDBZR" (id 1) (at 100.33 172.72 0)
+    (property "Value" "DRV5056A4" (id 1) (at 100.33 172.72 0)
       (effects (font (size 1.778 1.5113)) (justify left bottom))
     )
@@
       (effects (font (size 1.778 1.5113)) (justify left bottom))
     )
-    (property "Value" "DRV5057A1QDBZR" (id 1) (at 100.33 198.12 0)
+    (property "Value" "DRV5056A4" (id 1) (at 100.33 198.12 0)
       (effects (font (size 1.778 1.5113)) (justify left bottom))
     )
@@
     )
     (path "/c18c547b-8fb6-465c-8d4f-f47955f18040"
-      (reference "C3") (unit 1) (value "C-EUC0402") (footprint "Capacitor_SMD:C_0402_1005Metric_Pad0.74x0.62mm_HandSolder")
+      (reference "C3") (unit 1) (value "100nF") (footprint "Capacitor_SMD:C_0402_1005Metric_Pad0.74x0.62mm_HandSolder")
     )
     (path "/5c0ccebe-679d-484d-b15b-43f7d57dfe85"
-      (reference "C4") (unit 1) (value "C-EUC0402") (footprint "Capacitor_SMD:C_0402_1005Metric_Pad0.74x0.62mm_HandSolder")
+      (reference "C4") (unit 1) (value "100nF") (footprint "Capacitor_SMD:C_0402_1005Metric_Pad0.74x0.62mm_HandSolder")
     )
     (path "/822552ff-ff15-4eab-86bb-eac119fb8de4"
-      (reference "C5") (unit 1) (value "C-EUC0402") (footprint "Capacitor_SMD:C_0402_1005Metric_Pad0.74x0.62mm_HandSolder")
+      (reference "C5") (unit 1) (value "100nF") (footprint "Capacitor_SMD:C_0402_1005Metric_Pad0.74x0.62mm_HandSolder")
     )
     (path "/46c6a9b0-68b0-4697-b836-a3e7d4360485"
-      (reference "C6") (unit 1) (value "C-EUC0402") (footprint "Capacitor_SMD:C_0402_1005Metric_Pad0.74x0.62mm_HandSolder")
+      (reference "C6") (unit 1) (value "100nF") (footprint "Capacitor_SMD:C_0402_1005Metric_Pad0.74x0.62mm_HandSolder")
     )
     (path "/6494dd25-65d2-4517-88aa-8c88f41b35e6"
@@
     )
     (path "/3fe5e716-1781-447b-8b65-b39786c9a8c7"
-      (reference "U2") (unit 1) (value "DRV5057A1QDBZR") (footprint "TACTILE_28UFQFPN_SPI_v2.0:SOT23-BEC")
+      (reference "U2") (unit 1) (value "DRV5056A4") (footprint "TACTILE_28UFQFPN_SPI_v2.0:SOT23-BEC")
     )
     (path "/6492a9c1-d855-46fa-bcc4-d002c50c6d36"
-      (reference "U3") (unit 1) (value "DRV5057A1QDBZR") (footprint "TACTILE_28UFQFPN_SPI_v2.0:SOT23-BEC")
+      (reference "U3") (unit 1) (value "DRV5056A4") (footprint "TACTILE_28UFQFPN_SPI_v2.0:SOT23-BEC")
     )
     (path "/13bb8511-f982-481a-a66d-c5d6e0780f5b"
-      (reference "U4") (unit 1) (value "DRV5057A1QDBZR") (footprint "TACTILE_28UFQFPN_SPI_v2.0:SOT23-BEC")
+      (reference "U4") (unit 1) (value "DRV5056A4") (footprint "TACTILE_28UFQFPN_SPI_v2.0:SOT23-BEC")
     )
     (path "/49e9ca83-3b63-4ec8-8aaa-141f2730d80d"
-      (reference "U5") (unit 1) (value "DRV5057A1QDBZR") (footprint "TACTILE_28UFQFPN_SPI_v2.0:SOT23-BEC")
-    )
-  )
+      (reference "U5") (unit 1) (value "DRV5056A4") (footprint "TACTILE_28UFQFPN_SPI_v2.0:SOT23-BEC")
+    )
+  )
