File: UNIVERSAL_HALL_PCB_v2.8/universal_hall_pcb_v2.8.kicad_pcb (KiCad board)
At the start: 2 copper layers, 23.3 x 49.9 mm, 6 parts, among them J1 Conn_02x03_Odd_Even, J2 Conn_02x03_Odd_Even, U1 MA310

Commit message: add gripper and so on
Other:
- outline, holes or cut-outs redrawn
Changed lines of the file:
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@@
     (property "Sheetname" "")
     (attr through_hole)
-    (fp_text reference "J2" (at 2.769052 -1.172096 3.17) (layer "F.SilkS")
+    (fp_text reference "J2" (at -5.950814 -1.054113 3.17) (layer "F.SilkS")
       (effects (font (size 1 1) (thickness 0.15)))
     )
@@
     (property "Sheetname" "")
     (attr through_hole)
-    (fp_text reference "J1" (at 2.74471 6.157643 -3.17) (layer "F.SilkS")
+    (fp_text reference "J1" (at -5.475922 6.012011 -3.17) (layer "F.SilkS")
       (effects (font (size 1 1) (thickness 0.15)))
     )
@@
     (property "Sheetname" "")
     (attr smd)
-    (fp_text reference "R1" (at 0.1 -1.7) (layer "F.SilkS")
+    (fp_text reference "R1" (at 2.9 0.1) (layer "F.SilkS")
       (effects (font (size 1 1) (thickness 0.15)))
     )
@@
     (property "Sheetname" "")
     (attr through_hole)
-    (fp_text reference "TH1" (at -2.3 0.1) (layer "B.SilkS")
+    (fp_text reference "TH1" (at 5.15 0.1) (layer "B.SilkS")
       (effects (font (size 1 1) (thickness 0.15)) (justify mirror))
     )
@@
   )
   (gr_circle (center 174.1 84) (end 174.1 84) (layer "F.Adhes") (width 0.15) (fill none))
+  (gr_rect (start 182.5 106.3) (end 188.3 115.5) (layer "F.SilkS") (width 0.15) (fill solid))
+  (gr_rect (start 167.3 115.5) (end 188.3 127.8) (layer "F.SilkS") (width 0.15) (fill solid))
+  (gr_rect (start 164.7 77) (end 185.7 89.8) (layer "F.SilkS") (width 0.15) (fill solid))
   (gr_line (start 175.025653 103.49816) (end 175.025653 106.49816) (layer "Dwgs.User") (width 0.25))
   (gr_circle (center 180.227009 99.274161) (end 180.727009 99.274161) (layer "Dwgs.User") (width 0.25) (fill none))
@@
   (gr_circle (center 177.691586 110.56975) (end 178.191586 110.56975) (layer "Dwgs.User") (width 0.25) (fill none))
   (gr_circle (center 177.539177 96.891146) (end 178.039177 96.891146) (layer "Dwgs.User") (width 0.25) (fill none))
+  (gr_circle (center 183.8 105) (end 184.3 105) (layer "Edge.Cuts") (width 0.01) (fill none))
+  (gr_arc (start 183.850624 123.717192) (mid 179.267591 127.135146) (end 173.721527 125.746701) (layer "Edge.Cuts") (width 0.25))
+  (gr_circle (center 175.012968 119.037894) (end 176.512968 119.037894) (layer "Edge.Cuts") (width 0.25) (fill none))
+  (gr_arc (start 179.577049 79.816335) (mid 186.161398 91.523387) (end 188.499218 104.750001) (layer "Edge.Cuts") (width 0.25))
+  (gr_arc (start 165.768281 86.922212) (mid 165.153338 85.595855) (end 165.605163 84.205448) (layer "Edge.Cuts") (width 0.25))
   (gr_arc (start 188.499218 105.249998) (mid 187.289934 114.764268) (end 183.850625 123.717192) (layer "Edge.Cuts") (width 0.25))
+  (gr_arc (start 165.768281 86.922211) (mid 173.382382 102.577798) (end 168.93064 119.407947) (layer "Edge.Cuts") (width 0.25))
+  (gr_arc (start 188.499219 105.249999) (mid 188.25 105) (end 188.499218 104.750001) (layer "Edge.Cuts") (width 0.25))
+  (gr_circle (center 171.807787 86.112251) (end 173.307787 86.112251) (layer "Edge.Cuts") (width 0.25) (fill none))
+  (gr_line (start 169.246701 79.778472) (end 165.605163 84.205448) (layer "Edge.Cuts") (width 0.25))
   (gr_arc (start 169.246702 79.778472) (mid 174.420858 77.346455) (end 179.577049 79.816334) (layer "Edge.Cuts") (width 0.25))
-  (gr_arc (start 188.499219 105.249999) (mid 188.25 105) (end 188.499218 104.750001) (layer "Edge.Cuts") (width 0.25))
-  (gr_arc (start 179.577049 79.816335) (mid 186.161398 91.523387) (end 188.499218 104.750001) (layer "Edge.Cuts") (width 0.25))
-  (gr_line (start 169.246701 79.778472) (end 165.605163 84.205448) (layer "Edge.Cuts") (width 0.25))
-  (gr_circle (center 171.807787 86.112251) (end 173.307787 86.112251) (layer "Edge.Cuts") (width 0.25) (fill none))
-  (gr_arc (start 165.768281 86.922211) (mid 173.382382 102.577798) (end 168.93064 119.407947) (layer "Edge.Cuts") (width 0.25))
-  (gr_arc (start 183.850624 123.717192) (mid 179.267591 127.135146) (end 173.721527 125.746701) (layer "Edge.Cuts") (width 0.25))
+  (gr_line (start 173.721527 125.746701) (end 169.294551 122.105163) (layer "Edge.Cuts") (width 0.25))
   (gr_arc (start 169.294551 122.105163) (mid 168.58305 120.828002) (end 168.93064 119.407947) (layer "Edge.Cuts") (width 0.25))
-  (gr_circle (center 175.012968 119.037894) (end 176.512968 119.037894) (layer "Edge.Cuts") (width 0.25) (fill none))
-  (gr_line (start 173.721527 125.746701) (end 169.294551 122.105163) (layer "Edge.Cuts") (width 0.25))
-  (gr_arc (start 165.768281 86.922212) (mid 165.153338 85.595855) (end 165.605163 84.205448) (layer "Edge.Cuts") (width 0.25))
   (gr_line (start 0 210) (end 297 0) (layer "User.1") (width 0.15))
   (gr_line (start 0 0) (end 297 210) (layer "User.1") (width 0.15))
@@
     (effects (font (size 1.1 1.1) (thickness 0.275)))
   )
-  (gr_text "" (at 165.149744 135.535092) (layer "Edge.Cuts")
-    (effects (font (size 4.83362 3.04518) (thickness 0.604202)) (justify left top))
-  )
-  (gr_text "Produkt SOLIDWORKS Educational." (at 165.149744 128.284662) (layer "Edge.Cuts")
-    (effects (font (size 4.83362 3.04518) (thickness 0.604202)) (justify left top))
-  )
   (gr_text "Produkt SOLIDWORKS Educational." (at 163.238678 126.057027) (layer "User.2")
     (effects (font (size 4.83362 3.04518) (thickness 0.604202)) (justify left top))
@@
   (segment (start 185.3 104.75) (end 185.05 105) (width 0.2) (layer "F.Cu") (net 4))
   (segment (start 185.3 101.9) (end 185.3 104.75) (width 0.2) (layer "F.Cu") (net 4))
-  (segment (start 182 111.4) (end 182 108.05) (width 0.2) (layer "B.Cu") (net 4))
-  (segment (start 182 108.05) (end 185.05 105) (width 0.2) (layer "B.Cu") (net 4))
+  (segment (start 180.119083 113.272227) (end 180.127773 113.272227) (width 0.2) (layer "B.Cu") (net 4))
+  (segment (start 185.05 105.85) (end 185.05 105) (width 0.2) (layer "B.Cu") (net 4))
   (segment (start 180.127773 113.272227) (end 182 111.4) (width 0.2) (layer "B.Cu") (net 4))
-  (segment (start 180.119083 113.272227) (end 180.127773 113.272227) (width 0.2) (layer "B.Cu") (net 4))
+  (segment (start 182 108.9) (end 185.05 105.85) (width 0.2) (layer "B.Cu") (net 4))
+  (segment (start 182 111.4) (end 182 108.9) (width 0.2) (layer "B.Cu") (net 4))
   (segment (start 178.05 105.25) (end 178.613878 105.813878) (width 0.2) (layer "B.Cu") (net 5))
   (segment (start 177.0875 105.25) (end 178.05 105.25) (width 0.2) (layer "B.Cu") (net 5))
@@
   (segment (start 176.35 103.5125) (end 176.35 103.430918) (width 0.25) (layer "B.Cu") (net 12))
   (zone (net 6) (net_name "GND") (layers F&B.Cu) (hatch edge 0.508)
-    (connect_pads yes (clearance 0.508))
+    (connect_pads yes (clearance 0.1))
     (min_thickness 0.254) (filled_areas_thickness no)
     (fill yes (thermal_gap 0.508) (thermal_bridge_width 0.508))
@@
         (xy 168.1 80.8)
       )
-    )
-  )
-  (group "" (id 5cc35b56-06a9-4a47-adca-bfef757cb817)
-    (members
-      0658e700-f76e-4575-940d-28098c8b38a6
-      1056a7f0-3f20-4430-be76-49f3b0add7d1
-      1505b392-cb84-456b-b557-734e4111ee66
-      16994ac8-032f-4ecc-be8e-766efb4d858d
-      41334186-3118-4358-a1b3-e1b7823f7739
-      a1d6859a-c895-46a6-b5fd-133ffb4604a6
-      a65819fa-ef2a-4ecd-9a41-ca44fc29f55a
-      a6752cac-ef69-46a5-945a-806cf8cb0bed
-      af1c180f-225e-4620-a639-9a9825b441ef
-      bc40736e-91eb-48a9-8800-928c89d2f2a8
-      c5ce6437-2136-403e-ab3f-f0a853fdf7d8
-      eaff4267-8591-473a-9816-33f7bf30dac2
-      edb79f7b-8195-44ba-8877-ed2cecd3f6cc
-      f5594665-59c5-498e-9497-fdb14ce68db8
     )
   )
@@
     )
   )
+  (group "" (id f1eaf80c-1d6e-4263-a236-b4ec3ec76274)
+    (members
+      1ecaf9f2-ce7b-4b58-903a-48dc48ed33aa
+      2ba0089a-938a-4875-88f1-57a17f7fa0a7
+      34164b55-9dff-4742-ab9b-d81c08aaf77a
+      39139c3e-bcc1-494b-8506-3631e4547d6d
+      88d0c2e7-462d-44a2-9756-2ad1d898ee9e
+      9a9ad497-39bb-4a39-bf5c-f8dc47ce240c
+      a784a7c7-dac9-47f9-a810-c5a12d08ae52
+      b31946d9-7139-4b39-915f-23b19477ba9c
+      b6077c89-196c-4cf9-b8c7-6fe6cf576a32
+      de8bc0d3-1149-46f5-8154-6f9de78ebb3a
+      e681d574-7003-4f67-b68f-b630dce11190
+      f8e26a94-e9cd-4146-9274-17e961a1968b
+    )
+  )
