File: TACTILE_28UFQFPN_SPI_v2.1/TACTILE_28UFQFPN_SPI_v2.1.kicad_sch (KiCad schematic)
At the start: 20 parts, among them J1 59453-061110ECHLF, J2 59453-061110ECHLF, U1 STM32G071G8U6N, U2 DRV5056A4, U3 DRV5056A4, U4 DRV5056A4, U5 DRV5056A4

Commit message: tactile 2.1
Parts:
- removed PAD1, PAD2, PAD3, PAD4, PAD5: WIREPADSMD1,27-254, TACTILE_28UFQFPN_SPI_v2.0:SMD1,27-2,54, symbol Magnetic Finger SMALL Ampherol 28pin-eagle-import:WIREPADSMD1,27-254
- added J3: Conn_01x04_Male, footprints:PinHeader_1x04_P2.54mm_Vertical, symbol Connector:Conn_01x04_Male
- C1, C2, C3, C4, C5, C6: footprint Capacitor_SMD:C_0402_1005Metric_Pad0.74x0.62mm_HandSolder -> footprints:C_0603_1608Metric_Pad1.08x0.95mm_HandSolder
Connections:
- net 3V3: now also J3.4 (Pin_4)
- net GND: now also J3.3 (Pin_3)
- net SWCLK: now also J3.1 (Pin_1)
- net SWDIO: now also J3.2 (Pin_2)
