File: TACTILE_28UFQFPN_SPI_v2.1/TACTILE_28UFQFPN_SPI_v2.1.kicad_pcb (KiCad board)
At the start: 2 copper layers, 20 x 32 mm, 20 parts, among them J1 59453-061110ECHLF, J2 59453-061110ECHLF, U1 STM32G071G8U6N, U2 DRV5056A4, U3 DRV5056A4, U4 DRV5056A4, U5 DRV5056A4

Commit message: tactile 2.1
Parts:
- removed PAD1, PAD2, PAD3, PAD4, PAD5: WIREPADSMD1,27-254, TACTILE_28UFQFPN_SPI_v2.0:SMD1,27-2,54
- added J3: n.m., footprints:PinHeader_1x04_P2.54mm_Vertical, F.Cu at (154.8, 97.2)
- C1, C2, C3, C4, C5, C6: footprint Capacitor_SMD:C_0402_1005Metric_Pad0.74x0.62mm_HandSolder -> footprints:C_0603_1608Metric_Pad1.08x0.95mm_HandSolder
- JP1: footprint footprints:SolderJumper-2_P1.3mm_Bridged_Pad1.0x1.5mm -> footprints:SolderJumper-2_P1.3mm_Open_Pad1.0x1.5mm
- moved C1 7.93 mm to (155.0, 108.4), turned to 90 degrees
- moved C6 5.50 mm to (157.0, 117.6), turned to 90 degrees
- moved L1 4.73 mm to (145.4, 111.0), turned to 90 degrees
- moved J2 4.63 mm to (147.3, 100.1)
- moved J1 4.58 mm to (149.8, 109.9)
- moved JP1 1.50 mm to (152.1, 99.0), turned to -90 degrees
- moved C2 0.30 mm to (156.5, 108.4)
- moved C4 0.22 mm to (143.0, 94.4)
- moved C5 0.20 mm to (153.9, 94.4)
- moved C3 0.05 mm to (143.7, 115.7)
Routing:
- net /RST: track 8.15 -> 0.86 mm, vias 2 -> 1
- net /SPI_SCK: track 36.4 -> 43.4 mm, vias 2 -> 6
- net /3V3: track 40.6 -> 34.3 mm, vias 0 -> 4
- net GND: track 16.5 -> 10.4 mm, vias 21 -> 29
- net /SPI_MISO: track 39.4 -> 43.5 mm, vias 4 -> 2
- net /SPI_MOSI: track 6.50 -> 10.6 mm
- net /PASS_TRU: track 34.0 -> 38.0 mm, vias 2 -> 4
- net VCC: track 73.4 -> 76.2 mm, vias 5 -> 4
- net /SWDIO: track 14.7 -> 16.1 mm, vias 2 -> 1
- net /SWCLK: track 18.7 -> 20.0 mm
- net /SPI_CS: track 38.4 -> 39.6 mm
Other:
- outline, holes or cut-outs redrawn

Commit message: MASTER UPDATE v2
Other:
- board text added: "GRUBOŚĆ PCB = 0,6mm"
Changed lines of the file:
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@@
     (property "Sheetname" "")
     (attr smd)
-    (fp_text reference "C1" (at 2 6.4 180) (layer "F.SilkS")
+    (fp_text reference "C1" (at 0.9 2.8 270) (layer "F.SilkS")
       (effects (font (size 1 1) (thickness 0.15)))
     )
@@
     (property "Sheetname" "")
     (attr exclude_from_pos_files exclude_from_bom)
-    (fp_text reference "JP1" (at 0 -1.8 -90) (layer "F.SilkS")
+    (fp_text reference "JP1" (at -2.6 0) (layer "F.SilkS")
       (effects (font (size 1 1) (thickness 0.15)))
     )
@@
     (property "Sheetname" "")
     (attr through_hole)
-    (fp_text reference "J3" (at 0.8 -2.5) (layer "F.SilkS")
+    (fp_text reference "J3" (at 1.8 -2.8) (layer "F.SilkS")
       (effects (font (size 1 1) (thickness 0.15)))
     )
@@
       (effects (font (size 1 1) (thickness 0.15)))
     )
-    (fp_text user "*" (at -2.979674 -2.13233 -90) (layer "F.SilkS")
+    (fp_text user "*" (at -2.2536 -2.5489 -90) (layer "F.SilkS")
       (effects (font (size 1 1) (thickness 0.15)))
     )
@@
     (property "Sheetname" "")
     (attr smd)
-    (fp_text reference "C2" (at 0 4.2 90) (layer "F.SilkS")
+    (fp_text reference "C2" (at -1.3 1.3 90) (layer "F.SilkS")
       (effects (font (size 1 1) (thickness 0.15)))
     )
@@
     (fp_line (start -0.8 0.4) (end -0.8 -0.4) (layer "F.Fab") (width 0.1))
     (pad "1" smd roundrect locked (at -0.8625 0 90) (size 1.075 0.95) (layers "F.Cu" "F.Paste" "F.Mask") (roundrect_rratio 0.25)
-      (net 1 "VCC") (pinfunction "1") (pintype "passive"))
+      (net 1 "VCC") (pinfunction "1"))
     (pad "2" smd roundrect locked (at 0.8625 0 90) (size 1.075 0.95) (layers "F.Cu" "F.Paste" "F.Mask") (roundrect_rratio 0.25)
-      (net 2 "GND") (pinfunction "2") (pintype "passive"))
+      (net 2 "GND") (pinfunction "2"))
     (model "${KIPRJMOD}/../common_libraries/3dmodels/C_0603_1608Metric.step"
       (offset (xyz 0 0 0))
@@
     (effects (font (size 0.747776 0.747776) (thickness 0.065024)) (justify left bottom))
   )
+  (gr_text "GRUBOŚĆ PCB = 0,6mm" (at 139.7 131.4) (layer "Cmts.User")
+    (effects (font (size 5 5) (thickness 0.3)))
+  )
   (segment (start 153.803811 117.700889) (end 155.1011 118.998178) (width 0.1524) (layer "F.Cu") (net 1))
