File: IR_LED_PROJECTOR_v0.3/ir_led_projector_v0.3.kicad_sch (KiCad schematic)
At the start: 27 parts, among them Q1 Q_NMOS_DGS, U1 AZ1084-ADJ

Commit message: MASTER UPDATE
Parts:
- Q1: value Q_NMOS_DGS -> AON3402
Changed lines of the file:
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@@
       (effects (font (size 1.27 1.27)) (justify left))
     )
-    (property "Value" "Q_NMOS_DGS" (id 1) (at 181.61 100.9649 0)
+    (property "Value" "AON3402" (id 1) (at 181.61 100.9649 0)
       (effects (font (size 1.27 1.27)) (justify left))
     )
@@
     )
     (path "/10dc7bbf-0815-4851-9f11-c5ef255e8d9b"
-      (reference "Q1") (unit 1) (value "Q_NMOS_DGS") (footprint "IR_LED_PROJECTOR:DFN3x3A_8L_NEP_P")
+      (reference "Q1") (unit 1) (value "AON3402") (footprint "IR_LED_PROJECTOR:DFN3x3A_8L_NEP_P")
     )
     (path "/dc09fd24-3a59-4a3b-a68c-672e8a7575f8"
