File: UNIVERSAL_JOINT_v3_1/UNIVERSAL_JOINT_v3_1.kicad_pcb (KiCad board)
At the start: 2 copper layers, 76 x 75.9 mm, 142 parts, among them J10 HEADER_MALE_2X3_2.54_SMT, J11 Conn_02x05_Counter_Clockwise, J9 HEADER_MALE_2X3_2.54_SMT, Q1 STL110N10F7, Q2 STL110N10F7, Q201 BC856BWT1G, Q202 NVMFS4C03N, Q3 STL110N10F7, Q4 STL110N10F7, Q5 STL110N10F7, Q6 STL110N10F7, SW3 SW_MEC_5E, U1 STSPIN32G4, U2 TCAN332G, U6 MA730, X1 Crystal_GND24_Small

Commit message: UJ 3.1 IR 0.3 TACTILE 2.1
Parts:
- removed C22, C23, C24: N.M., footprints:C_0603_1608Metric_Pad1.08x0.95mm_HandSolder
- removed C33: 220uF 100V, footprints:CP_Radial_D6.3mm_P2.50mm
- removed J11: Conn_02x05_Counter_Clockwise, Connector:Tag-Connect_TC2070-IDC-FP_2x07_P1.27mm_Vertical
- removed R1, R10, R11, R12, R22, R23, R24: 0, footprints:R_0603_1608Metric_Pad0.98x0.95mm_HandSolder
- removed R16, R17, R18, R28, R29, R30: N.M., footprints:R_0603_1608Metric_Pad0.98x0.95mm_HandSolder
- added D206: RED, footprints:D_0603_1608Metric_Pad1.05x0.95mm_HandSolder, F.Cu at (170.0, 95.3)
- added D207: ORANGE, footprints:D_0603_1608Metric_Pad1.05x0.95mm_HandSolder, F.Cu at (153.1, 71.4)
- added D208: GREEN, footprints:D_0603_1608Metric_Pad1.05x0.95mm_HandSolder, F.Cu at (168.4, 98.6)
- added J12: FTSH-107-01-L-DV-K-TR, UNIVERSAL_JOINT:SAMTEC_FTSH-107-01-L-DV-K-TR, F.Cu at (148.5, 138.0)
- added JP1: SolderJumper_2_Open, footprints:SolderJumper-2_P1.3mm_Open_TrianglePad1.0x1.5mm, F.Cu at (137.0, 130.6)
- added JP2: SolderJumper_2_Open, footprints:SolderJumper-2_P1.3mm_Open_TrianglePad1.0x1.5mm, F.Cu at (137.0, 133.2)
- added JP3: SolderJumper_2_Open, footprints:SolderJumper-2_P1.3mm_Open_TrianglePad1.0x1.5mm, F.Cu at (137.0, 135.8)
- added JP4: SolderJumper_2_Open, footprints:SolderJumper-2_P1.3mm_Open_TrianglePad1.0x1.5mm, F.Cu at (137.0, 138.4)
- added NT1: NetTie_2, footprints:NetTie-2_SMD_Pad0.5mm, F.Cu at (168.7, 75.7)
- added Q203: 2PC4081S,115, UNIVERSAL_JOINT:SOT23-EBC, F.Cu at (173.5, 98.1)
- added R206: 5,23k, footprints:R_0603_1608Metric_Pad0.98x0.95mm_HandSolder, F.Cu at (167.4, 96.1)
- added R207: 13,7k, footprints:R_0603_1608Metric_Pad0.98x0.95mm_HandSolder, F.Cu at (168.4, 100.2)
- added R208: 200R, footprints:R_0603_1608Metric_Pad0.98x0.95mm_HandSolder, F.Cu at (173.6, 90.0)
- added R209: 130R, footprints:R_0603_1608Metric_Pad0.98x0.95mm_HandSolder, F.Cu at (173.6, 91.6)
- added R210: 200R, footprints:R_0603_1608Metric_Pad0.98x0.95mm_HandSolder, F.Cu at (173.6, 95.3)
- added R211: 4.6k, footprints:R_0603_1608Metric_Pad0.98x0.95mm_HandSolder, F.Cu at (154.8, 71.4)
- added R212: 80R, footprints:R_0603_1608Metric_Pad0.98x0.95mm_HandSolder, F.Cu at (170.0, 97.0)
- added R213: 100k, footprints:R_0603_1608Metric_Pad0.98x0.95mm_HandSolder, F.Cu at (140.4, 135.0)
- added R214: 100k, footprints:R_0603_1608Metric_Pad0.98x0.95mm_HandSolder, F.Cu at (140.4, 136.5)
- added R215: 100k, footprints:R_0603_1608Metric_Pad0.98x0.95mm_HandSolder, F.Cu at (140.4, 138.0)
- added R216: 100k, footprints:R_0603_1608Metric_Pad0.98x0.95mm_HandSolder, F.Cu at (140.4, 139.5)
- added TP14: TestPoint, footprints:Pin_D1.2mm_L10.2mm_W2.9mm_FlatFork, F.Cu at (171.0, 103.0)
- added TP15: TestPoint, footprints:Pin_D1.2mm_L10.2mm_W2.9mm_FlatFork, F.Cu at (166.0, 103.0)
- added TP16: GND, footprints:Pin_D1.2mm_L10.2mm_W2.9mm_FlatFork, F.Cu at (128.8, 131.2)
- added TP17: GND, footprints:Pin_D1.2mm_L10.2mm_W2.9mm_FlatFork, F.Cu at (124.0, 131.2)
- added TP18: TestPoint_Small, footprints:TestPoint_Pad_1.0x1.0mm, F.Cu at (154.2, 95.0)
- added TP19: TestPoint_Small, footprints:TestPoint_Pad_1.0x1.0mm, F.Cu at (156.3, 95.0)
- added TP20: TestPoint_Small, footprints:TestPoint_Pad_1.0x1.0mm, F.Cu at (158.4, 95.0)
- added TP21: TestPoint_Small, footprints:TestPoint_Pad_1.0x1.0mm, F.Cu at (162.6, 95.0)
- added TP22: TestPoint_Small, footprints:TestPoint_Pad_1.0x1.0mm, F.Cu at (160.5, 95.0)
- added TP23: TestPoint_Small, footprints:TestPoint_Pad_1.0x1.0mm, F.Cu at (164.7, 95.0)
- C31, C32: value 220uF 100V -> 330uF 100V; footprint footprints:CP_Radial_D6.3mm_P2.50mm -> footprints:CP_Radial_D12.5mm_P5.00mm
- D201: value LEDCHIP-LED0603 -> GREEN; footprint UNIVERSAL_JOINT_v2_1:CHIP-LED0603 -> footprints:D_0603_1608Metric_Pad1.05x0.95mm_HandSolder
- D203: footprint UNIVERSAL_JOINT_v2_1:DPACK -> UNIVERSAL_JOINT:DPACK
- D204: footprint UNIVERSAL_JOINT_v2_1:SOD123 -> footprints:D_SOD-123
- D205: value ZENER-DIODESOT23 -> ACZRW5242B-G; footprint Package_TO_SOT_SMD:TO-252-2 -> footprints:D_SOD-123; moved to F.Cu
- J10: value HEADER_MALE_2X3_2.54_SMT -> N.M.
- Q1, Q2, Q3, Q4, Q5, Q6: value STL110N10F7 -> IAUC120N06S5L; footprint footprints:STL110N10F7 -> ST:STL110N10F7
- Q201: footprint UNIVERSAL_JOINT_v2_1:SOT23 -> UNIVERSAL_JOINT:SOT23
- Q202: value NVMFS4C03N -> IAUC120N06S5L; footprint footprints:STL110N10F7 -> ST:STL110N10F7; moved to B.Cu
- R205: footprint footprints:R_0603_1608Metric_Pad0.98x0.95mm_HandSolder -> UNIVERSAL_JOINT:DPACK; moved to B.Cu
- SW3: footprint Button_Switch_SMD:Panasonic_EVQPUJ_EVQPUA -> UNIVERSAL_JOINT:SKHUALE010
- TP1, TP11, TP12, TP13, TP2, TP3, TP4: footprint footprints:Pin_D1.2mm_L10.2mm_W2.9mm_FlatFork -> UNIVERSAL_JOINT:1-726388-2
- TP10, TP7, TP8, TP9: footprint footprints:Pin_D0.7mm_L6.5mm_W1.8mm_FlatFork -> footprints:Pin_D1.2mm_L10.2mm_W2.9mm_FlatFork
- U1: value STSPIN32G4 -> QFN_IN32G4_STM; footprint footprints:STSPIN32G4 -> UNIVERSAL_JOINT:STSPIN32G4
- moved C10 88.5 mm to (138.4, 120.1)
- moved C8 84.1 mm to (138.4, 123.3)
- moved R9 81.6 mm to (140.9, 121.0), turned to 90 degrees
- moved C11 76.5 mm to (138.4, 118.5)
- moved C9 75.3 mm to (138.4, 121.8)
- moved R6 71.4 mm to (154.5, 134.4), turned to 90 degrees
- moved D205 69.0 mm to (150.8, 79.2), turned to 90 degrees
- moved C6 62.7 mm to (158.9, 135.3), turned to 180 degrees
- moved C2 61.3 mm to (114.7, 117.7), turned to 90 degrees
- moved R7 60.8 mm to (156.3, 132.9), turned to 90 degrees
- moved C7 58.5 mm to (158.9, 133.7), turned to 180 degrees
- moved SW3 58.1 mm to (172.4, 84.1)
- moved R8 55.9 mm to (161.2, 129.5), turned to 90 degrees
- moved D202 54.0 mm to (144.3, 75.3), turned to -90 degrees
- moved C12 53.9 mm to (158.9, 132.0), turned to 180 degrees
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Connections:
- C13 pad 1: GND -> GNDPWR
- C14 pad 1: GND -> GNDPWR
- C15 pad 1: GND -> GNDPWR
- C19 pad 2: /COMP3 -> /VBUS
- C31 pad 1: /48V -> VM
- C31 pad 2: GND -> GNDPWR
- C32 pad 1: /48V -> VM
- C32 pad 2: GND -> GNDPWR
- D2 pad 2: Net-(D2-Pad2) -> /GHS1_MOS
- D202 pad 2: GND -> GNDPWR
- D205 pad 1: GND -> Net-(D205-Pad1)
- D205 pad 2: (no net) -> GNDPWR
- D3 pad 2: Net-(D3-Pad2) -> /GHS2_MOS
- D4 pad 2: Net-(D4-Pad2) -> /GHS3_MOS
- D5 pad 2: Net-(D5-Pad2) -> /GLS1_MOS
- D6 pad 2: Net-(D6-Pad2) -> /GLS2_MOS
- D7 pad 2: Net-(D7-Pad2) -> /GLS3_MOS
- D8 pad 2: /COMP3 -> /VBUS
- J10 pad 1: unconnected-(J10-Pad1) -> /MGL
- J10 pad 2: unconnected-(J10-Pad2) -> /SPI_SCK
- J10 pad 3: unconnected-(J10-Pad3) -> /SPI_MISO
- J10 pad 4: unconnected-(J10-Pad4) -> /SPI_MOSI
- J10 pad 5: unconnected-(J10-Pad5) -> /MA710_CS
- J10 pad 6: unconnected-(J10-Pad6) -> /MGH
- J9 pad 1: unconnected-(J9-Pad1) -> GND
- J9 pad 2: unconnected-(J9-Pad2) -> /BEARING_TEMP
- J9 pad 3: unconnected-(J9-Pad3) -> /B
- J9 pad 4: unconnected-(J9-Pad4) -> /A
- Q1 pad 4: Net-(Q1-Pad4) -> /GHS1_MOS
- Q2 pad 4: Net-(Q2-Pad4) -> /GHS2_MOS
- Q201 pad 1: Net-(D204-PadANODE) -> Net-(D204-Pad2)
- Q202 pad 1: (no net) -> GNDPWR
- Q202 pad 2: (no net) -> GNDPWR
- Q202 pad 3: (no net) -> GNDPWR
- Q202 pad 4: (no net) -> Net-(D205-Pad1)
- Q202 pad 5: (no net) -> Net-(Q202-Pad5)
- Q202 pad 6: (no net) -> Net-(Q202-Pad5)
- Q202 pad 7: (no net) -> Net-(Q202-Pad5)
- Q202 pad 8: (no net) -> Net-(Q202-Pad5)
- Q3 pad 4: Net-(Q3-Pad4) -> /GHS3_MOS
- Q4 pad 4: Net-(Q4-Pad4) -> /GLS1_MOS
- Q5 pad 4: Net-(Q5-Pad4) -> /GLS2_MOS
- Q6 pad 4: Net-(Q6-Pad4) -> /GLS3_MOS
- R13 pad 2: Net-(Q1-Pad4) -> /GHS1_MOS
- R14 pad 2: Net-(Q2-Pad4) -> /GHS2_MOS
- R15 pad 2: Net-(Q3-Pad4) -> /GHS3_MOS
- R201 pad 1: GND -> GNDPWR
- R201 pad 2: Net-(D201-PadC) -> Net-(D201-Pad1)
- R202 pad 1: Net-(D204-PadCATHODE) -> Net-(D204-Pad1)
- R203 pad 1: Net-(D205-Pad3) -> Net-(D205-Pad1)
- R204 pad 1: GND -> GNDPWR
- R204 pad 2: Net-(D205-Pad3) -> Net-(D205-Pad1)
- R205 pad 1: Net-(Q202-PadP$5) -> Net-(Q202-Pad5)
- R205 pad 2: VM -> GNDPWR
- R25 pad 2: Net-(Q4-Pad4) -> /GLS1_MOS
- R26 pad 2: Net-(Q5-Pad4) -> /GLS2_MOS
- R27 pad 2: Net-(Q6-Pad4) -> /GLS3_MOS
- R31 pad 2: GND -> GNDPWR
- R32 pad 2: GND -> GNDPWR
- R33 pad 2: GND -> GNDPWR
- R34 pad 2: GND -> GNDPWR
- R35 pad 2: GND -> GNDPWR
- R36 pad 2: GND -> GNDPWR
- R37 pad 1: /COMP3 -> /VBUS
- R39 pad 2: /COMP3 -> /VBUS
- R50 pad 1: GND -> GNDPWR
- R51 pad 1: GND -> GNDPWR
- R52 pad 1: GND -> GNDPWR
- TP3 pad 1: GND -> GNDPWR
- TP4 pad 1: GND -> GNDPWR
- U1 pad 12: unconnected-(U1-Pad12) -> /MA730_CS
- U1 pad 17: unconnected-(U1-Pad17) -> /BEARING_TEMP
- U1 pad 28: unconnected-(U1-Pad28) -> /TORQUE_CS
- U1 pad 3: unconnected-(U1-Pad3) -> /MA710_CS
- U1 pad 4: /CAN_SHDN -> /SEC_IN
- U1 pad 44: unconnected-(U1-Pad44) -> /DIP1
- U1 pad 5: unconnected-(U1-Pad5) -> /SEC_OUT
- U1 pad 53: unconnected-(U1-Pad53) -> /DIP4
- U1 pad 59: unconnected-(U1-Pad59) -> /DIP3
- U1 pad 60: unconnected-(U1-Pad60) -> /DIP2
- U6 pad 5: /CS1 -> /MA730_CS
Routing:
- net /VDD: track 14.7 -> 118.6 mm, vias 4 -> 5
- net /nRST: track 15.1 -> 78.3 mm, vias 2 -> 4
- net /SPI_MISO: track 17.4 -> 76.1 mm, vias 1 -> 5
- net Net-(Q1-Pad4): track 54.2 -> 0.00 mm, vias 2 -> 0
- net /SEC_OUT: track 0.00 -> 53.5 mm, vias 0 -> 2
- net /MA710_CS: track 0.00 -> 53.3 mm, vias 0 -> 3
- net /SPI_MOSI: track 15.5 -> 65.3 mm, vias 1 -> 4
- net VM: track 3.59 -> 50.6 mm, vias 190 -> 52
- net /SEC_IN: track 0.00 -> 44.7 mm, vias 0 -> 2
- net /TORQUE_CS: track 0.00 -> 41.2 mm, vias 0 -> 2
- net GNDPWR: track 0.00 -> 40.8 mm, vias 0 -> 90
- net Net-(Q2-Pad4): track 38.8 -> 0.00 mm, vias 2 -> 0
- net /BEARING_TEMP: track 0.00 -> 38.6 mm, vias 0 -> 3
- net /GHS1_MOS: track 0.00 -> 38.3 mm, vias 0 -> 2
- net /SPI_SCK: track 15.3 -> 52.1 mm, vias 1 -> 4
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- added copper zone on B.Cu, net GNDPWR
- added copper zone on F.Cu, net GNDPWR
- added copper zone on B.Cu, net Net-(Q202-Pad5)
- added copper zone on F.Cu, net Net-(Q202-Pad5)
Other:
- board text added: "*"
- board text added: "1"
- board text added: "12V"
- board text added: "2"
- board text added: "3"
- board text added: "4"
- board text added: "48V"
- board text added: "B"
- board text added: "GND"
- board text added: "H"
- board text added: "L"
- board text added: "PGND"
- board text added: "Produkt SOLIDWORKS Educational."
- board text added: "R"
- board text added: "S"
- board text added: "Y"
- board text added: "v3.1"

Commit message: add gripper and so on
Parts:
- J10, J9: footprint footprints:M207810345 -> UNIVERSAL_JOINT:M207810345
- R201: value 200 -> 4.5k
- R39: value 72.3k 1% -> 3.01k 1%
- SW3: value SW_MEC_5E -> SKHUALE010
- TP11, TP12, TP13: value TestPoint -> 1-726388-2

Commit message: update 3.1
Parts:
- TP10, TP14, TP15, TP16, TP17, TP5, TP6, TP7, TP8, TP9: footprint footprints:Pin_D1.2mm_L10.2mm_W2.9mm_FlatFork -> UNIVERSAL_JOINT:61-2348-11_0030
- U1: value QFN_IN32G4_STM -> STSPIN32G4

Commit message: update UJ 3.1 NM values
Parts:
- D203: value MBRD20 -> BRIDGED
- D204: value STPS0560Z -> NM
- D205: value ACZRW5242B-G -> NM
- D206: value RED -> NM
- D207: value ORANGE -> NM
- D208: value GREEN -> NM
- Q201: value BC856BWT1G -> NM
- Q202: value IAUC120N06S5L -> NM
- R202: value 10k -> NM
- R203, R204: value 200 -> NM
- R205: value 47R -> NM
- R209: value 130R -> NM
- R211: value 4.6k -> NM
- R212: value 80R -> NM
- X1: value Crystal_GND24_Small -> ECS-240-8-36B2-CKM-TR
Changed lines of the file:
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@@
       (effects (font (size 0.7 0.7) (thickness 0.15)))
     )
-    (fp_text value "4.6k" (at 0 1.43 90) (layer "F.Fab")
+    (fp_text value "NM" (at 0 1.43 90) (layer "F.Fab")
       (effects (font (size 0.8 0.8) (thickness 0.15)))
     )
@@
       (effects (font (size 0.7 0.7) (thickness 0.15)))
     )
-    (fp_text value "STPS0560Z" (at 0 2.1) (layer "F.Fab")
+    (fp_text value "NM" (at 0 2.1) (layer "F.Fab")
       (effects (font (size 1 1) (thickness 0.15)))
     )
@@
       (effects (font (size 0.7 0.7) (thickness 0.15)))
     )
-    (fp_text value "GREEN" (at 0 1.43) (layer "F.Fab")
+    (fp_text value "NM" (at 0 1.43) (layer "F.Fab")
       (effects (font (size 0.8 0.8) (thickness 0.15)))
     )
@@
       (effects (font (size 0.7 0.7) (thickness 0.15)))
     )
-    (fp_text value "Crystal_GND24_Small" (at 0 2.2) (layer "F.Fab")
+    (fp_text value "ECS-240-8-36B2-CKM-TR" (at 0 2.2) (layer "F.Fab")
       (effects (font (size 0.8 0.8) (thickness 0.15)))
     )
@@
       (effects (font (size 0.7 0.7) (thickness 0.15)))
     )
-    (fp_text value "200" (at 0 1.43) (layer "F.Fab")
+    (fp_text value "NM" (at 0 1.43) (layer "F.Fab")
       (effects (font (size 0.8 0.8) (thickness 0.15)))
     )
@@
       (effects (font (size 0.7 0.7) (thickness 0.15)) (justify left bottom))
     )
-    (fp_text value "BC856BWT1G" (at -1.905 3.175 -90) (layer "F.Fab")
+    (fp_text value "NM" (at -1.905 3.175 -90) (layer "F.Fab")
       (effects (font (size 0.8 0.8) (thickness 0.1016)) (justify left bottom))
     )
@@
       (effects (font (size 0.7 0.7) (thickness 0.15)))
     )
-    (fp_text value "130R" (at 0 1.43) (layer "F.Fab")
+    (fp_text value "NM" (at 0 1.43) (layer "F.Fab")
       (effects (font (size 0.8 0.8) (thickness 0.15)))
     )
@@
       (effects (font (size 0.7 0.7) (thickness 0.15)))
     )
-    (fp_text value "ORANGE" (at 0 1.43 90) (layer "F.Fab")
+    (fp_text value "NM" (at 0 1.43 90) (layer "F.Fab")
       (effects (font (size 0.8 0.8) (thickness 0.15)))
     )
@@
       (effects (font (size 0.7 0.7) (thickness 0.15)))
     )
-    (fp_text value "RED" (at 0 1.43) (layer "F.Fab")
+    (fp_text value "NM" (at 0 1.43) (layer "F.Fab")
       (effects (font (size 0.8 0.8) (thickness 0.15)))
     )
@@
       (effects (font (size 0.7 0.7) (thickness 0.15)))
     )
-    (fp_text value "ACZRW5242B-G" (at 0 2.1 90) (layer "F.Fab")
+    (fp_text value "NM" (at 0 2.1 90) (layer "F.Fab")
       (effects (font (size 0.8 0.8) (thickness 0.15)))
     )
@@
       (effects (font (size 0.7 0.7) (thickness 0.15)))
     )
-    (fp_text value "10k" (at 0 1.43 90) (layer "F.Fab")
+    (fp_text value "NM" (at 0 1.43 90) (layer "F.Fab")
       (effects (font (size 0.8 0.8) (thickness 0.15)))
     )
@@
       (effects (font (size 0.7 0.7) (thickness 0.15)))
     )
-    (fp_text value "80R" (at 0 1.43) (layer "F.Fab")
+    (fp_text value "NM" (at 0 1.43) (layer "F.Fab")
       (effects (font (size 0.8 0.8) (thickness 0.15)))
     )
@@
       (effects (font (size 0.7 0.7) (thickness 0.15)))
     )
-    (fp_text value "200" (at 0 1.43) (layer "F.Fab")
+    (fp_text value "NM" (at 0 1.43) (layer "F.Fab")
       (effects (font (size 0.8 0.8) (thickness 0.15)))
     )
@@
       (effects (font (size 0.8 0.8) (thickness 0.1016)) (justify left bottom mirror))
     )
-    (fp_text value "47R" (at 5.08 -2.54) (layer "B.Fab")
+    (fp_text value "NM" (at 5.08 -2.54) (layer "B.Fab")
       (effects (font (size 0.8 0.8) (thickness 0.1016)) (justify left bottom mirror))
     )
@@
       (effects (font (size 0.8 0.8) (thickness 0.15)) (justify mirror))
     )
-    (fp_text value "IAUC120N06S5L" (at 0 -3.9 90) (layer "Dwgs.User") hide
+    (fp_text value "NM" (at 0 -3.9 90) (layer "Dwgs.User") hide
       (effects (font (size 0.8 0.8) (thickness 0.15)))
     )
@@
       (effects (font (size 1.1684 1.1684) (thickness 0.1016)) (justify left bottom mirror))
     )
-    (fp_text value "MBRD20" (at 5.08 -2.54 90) (layer "B.Fab")
+    (fp_text value "BRIDGED" (at 5.08 -2.54 90) (layer "B.Fab")
       (effects (font (size 1.1684 1.1684) (thickness 0.1016)) (justify left bottom mirror))
     )

Commit message: MASTER UPDATE
Parts:
- R37: value 72.3k 1% -> 73.2k 1%
- U1: value STSPIN32G4 -> QFN_IN32G4_STM
