File: UNIVERSAL_JOINT_v3_1/UNIVERSAL_JOINT_v3_1.kicad_sch (KiCad schematic)
At the start: 142 parts, among them J10 HEADER_MALE_2X3_2.54_SMT, J11 Conn_02x05_Counter_Clockwise, J9 HEADER_MALE_2X3_2.54_SMT, Q1 STL110N10F7, Q2 STL110N10F7, Q201 BC856BWT1G, Q202 NVMFS4C03N, Q3 STL110N10F7, Q4 STL110N10F7, Q5 STL110N10F7, Q6 STL110N10F7, SW3 SW_MEC_5E, U1 STSPIN32G4, U2 TCAN332G, U6 MA730, X1 Crystal_GND24_Small

Commit message: UJ 3.1 IR 0.3 TACTILE 2.1
Parts:
- removed C22, C23, C24: N.M., footprints:C_0603_1608Metric_Pad1.08x0.95mm_HandSolder, symbol Device:C
- removed C33: 220uF 100V, footprints:CP_Radial_D6.3mm_P2.50mm, symbol Device:C_Polarized_Small
- removed D201: LEDCHIP-LED0603, UNIVERSAL_JOINT_v2_1:CHIP-LED0603, symbol import_z_eagle-eagle-import:LEDCHIP-LED0603
- removed D205: ZENER-DIODESOT23, Package_TO_SOT_SMD:TO-252-2, symbol import_z_eagle-eagle-import:ZENER-DIODESOT23
- removed J11: Conn_02x05_Counter_Clockwise, Connector:Tag-Connect_TC2070-IDC-FP_2x07_P1.27mm_Vertical, symbol Connector_Generic:Conn_02x07_Counter_Clockwise
- removed Q202: NVMFS4C03N, footprints:STL110N10F7, symbol import_z_eagle-eagle-import:NVMFS4C03N
- removed R10, R11, R12, R22, R23, R24: 0, footprints:R_0603_1608Metric_Pad0.98x0.95mm_HandSolder, symbol Device:R
- removed R16, R17, R18, R28, R29, R30: N.M., footprints:R_0603_1608Metric_Pad0.98x0.95mm_HandSolder, symbol Device:R
- removed R205: 47R, footprints:R_0603_1608Metric_Pad0.98x0.95mm_HandSolder, symbol Device:R
- added D201, D208: GREEN, footprints:D_0603_1608Metric_Pad1.05x0.95mm_HandSolder, symbol Device:LED
- added D205: ACZRW5242B-G, footprints:D_SOD-123, symbol Device:D_Zener
- added D206: RED, footprints:D_0603_1608Metric_Pad1.05x0.95mm_HandSolder, symbol Device:LED
- added D207: ORANGE, footprints:D_0603_1608Metric_Pad1.05x0.95mm_HandSolder, symbol Device:LED
- added J12: FTSH-107-01-L-DV-K-TR, UNIVERSAL_JOINT:SAMTEC_FTSH-107-01-L-DV-K-TR, symbol FTSH-107-01-L-DV-K-TR:FTSH-107-01-L-DV-K-TR
- added JP1, JP2, JP3, JP4: SolderJumper_2_Open, footprints:SolderJumper-2_P1.3mm_Open_TrianglePad1.0x1.5mm, symbol Jumper:SolderJumper_2_Open
- added NT1: NetTie_2, footprints:NetTie-2_SMD_Pad0.5mm, symbol Device:NetTie_2
- added Q202: IAUC120N06S5L, ST:STL110N10F7, symbol STL110N10F7:STL110N10F7
- added Q203: 2PC4081S,115, UNIVERSAL_JOINT:SOT23-EBC, symbol UNIVERSAL_JOINT_v2_1-eagle-import:-NPN-SOT23-EBC
- added R205: 47R, UNIVERSAL_JOINT:DPACK, symbol UNIVERSAL_JOINT_v2_1-eagle-import:PF2205-47RF1TO-202_HOT
- added R206: 5,23k, footprints:R_0603_1608Metric_Pad0.98x0.95mm_HandSolder, symbol Device:R
- added R207: 13,7k, footprints:R_0603_1608Metric_Pad0.98x0.95mm_HandSolder, symbol Device:R
- added R208, R210: 200R, footprints:R_0603_1608Metric_Pad0.98x0.95mm_HandSolder, symbol Device:R
- added R209: 130R, footprints:R_0603_1608Metric_Pad0.98x0.95mm_HandSolder, symbol Device:R
- added R211: 4.6k, footprints:R_0603_1608Metric_Pad0.98x0.95mm_HandSolder, symbol Device:R
- added R212: 80R, footprints:R_0603_1608Metric_Pad0.98x0.95mm_HandSolder, symbol Device:R
- added R213, R214, R215, R216: 100k, footprints:R_0603_1608Metric_Pad0.98x0.95mm_HandSolder, symbol Device:R
- added TP14, TP15: TestPoint, footprints:Pin_D1.2mm_L10.2mm_W2.9mm_FlatFork, symbol Connector:TestPoint
- added TP16, TP17: GND, footprints:Pin_D1.2mm_L10.2mm_W2.9mm_FlatFork, symbol Connector:TestPoint
- added TP18, TP19, TP20, TP21, TP22, TP23: TestPoint_Small, footprints:TestPoint_Pad_1.0x1.0mm, symbol Connector:TestPoint_Small
- C31, C32: value 220uF 100V -> 330uF 100V; footprint footprints:CP_Radial_D6.3mm_P2.50mm -> footprints:CP_Radial_D12.5mm_P5.00mm
- D203: footprint UNIVERSAL_JOINT_v2_1:DPACK -> UNIVERSAL_JOINT:DPACK
- D204: footprint UNIVERSAL_JOINT_v2_1:SOD123 -> footprints:D_SOD-123; symbol import_z_eagle-eagle-import:STPS0560Z -> Device:D_Schottky_Small
- J10: value HEADER_MALE_2X3_2.54_SMT -> N.M.
- Q1, Q2, Q3, Q4, Q5, Q6: value STL110N10F7 -> IAUC120N06S5L; footprint footprints:STL110N10F7 -> ST:STL110N10F7
- Q201: footprint UNIVERSAL_JOINT_v2_1:SOT23 -> UNIVERSAL_JOINT:SOT23
- R1: value 0 -> n.m
- SW3: footprint Button_Switch_SMD:Panasonic_EVQPUJ_EVQPUA -> UNIVERSAL_JOINT:SKHUALE010
- TP1, TP11, TP12, TP13, TP2, TP3, TP4: footprint footprints:Pin_D1.2mm_L10.2mm_W2.9mm_FlatFork -> UNIVERSAL_JOINT:1-726388-2
- TP10, TP7, TP8, TP9: footprint footprints:Pin_D0.7mm_L6.5mm_W1.8mm_FlatFork -> footprints:Pin_D1.2mm_L10.2mm_W2.9mm_FlatFork
- U1: footprint footprints:STSPIN32G4 -> UNIVERSAL_JOINT:STSPIN32G4
Connections:
- net COMP3 is gone; now on net VBUS: C19.2, D8.2 (A), R37.1, R39.2
- net CS1 is gone; now on net MA730_CS: U6.5 (~{CS})
- net 48V: now also D201.2 (A); no longer C31.1, C32.1
- net A: now also J9.4
- net B: now also J9.3
- net GND: now also J9.1, J12.05, J12.07, J12.11, JP1.2 (B), JP2.2 (B), JP3.2 (B), JP4.2 (B), NT1.1, R206.1, R209.2, R210.1, R212.2, TP16.1, TP17.1, TP18.1; no longer C13.1, C14.1, C15.1, C31.2, C32.2, D202.2 (A), R201.1, R204.1, R31.2, R32.2, R33.2, R34.2, R35.2, R36.2, R50.1, R51.1, R52.1, TP3.1, TP4.1
- net JTDI: now also J12.10
- net SPI_MISO: now also J10.3, TP21.1
- net SPI_MOSI: now also J10.4, TP23.1
- net SPI_SCK: now also J10.2, TP22.1
- net SWCLK/JTCK: now also J12.06, J12.09
- net SWDIO/JTMS: now also J12.04
- net SWO/JTDO: now also J12.08
- net UART_RX: now also J12.13
- net UART_TX: now also J12.14
- net VDD: now also R213.1, R214.1, R215.1, R216.1, TP19.1
- net VM: now also C31.1, C32.1, D207.2 (A), R205.3
- net nRST: now also J12.12
- net GLS3_MOS: now reaches D7.2 (A)
- net GLS3_MOS: now also Q6.4, R27.2
- net GLS1_MOS: now reaches Q4.4, R25.2
- net GLS1_MOS: now also D5.2 (A)
- net at Q201.1 (B): now also D204.2 (A); no longer D204.ANODE
- net GLS2_MOS: now reaches Q5.4, R26.2
- net GLS2_MOS: now also D6.2 (A)
- net at R201.2: now also D201.1 (K)
- net MA730_CS: now reaches U1.12 (PC3)
- net BEARING_TEMP: now reaches U1.17 (PA4)
- net BEARING_TEMP: now also J9.2
- net TORQUE_CS: now reaches U1.28 (PB10)
- net TORQUE_CS: now also TP20.1
- net MA710_CS: now reaches U1.3 (PC13)
- net MA710_CS: now also J10.5
- net DIP1: now reaches U1.44 (PA8)
- net DIP1: now also JP1.1 (A), R213.2
- net SEC_OUT: now reaches U1.5 (PC15)
- net SEC_OUT: now also R208.1
- net DIP4: now reaches U1.53 (PD2)
- net DIP4: now also JP4.1 (A), R216.2
- net DIP3: now reaches U1.59 (PB8)
- net DIP3: now also JP3.1 (A), R215.2
- net DIP2: now reaches U1.60 (PB9)
- net DIP2: now also JP2.1 (A), R214.2
- net GHS1_MOS: now reaches D2.2 (A)
- net GHS1_MOS: now also Q1.4, R13.2
- net at R203.1, R204.2: now also D205.1 (K), Q202.4
- net GHS2_MOS: now reaches D3.2 (A)
- net GHS2_MOS: now also Q2.4, R14.2
- net at R202.1: now also D204.1 (K); no longer D204.CATHODE
- net MGL: now reaches J10.1
- net MGH: now reaches J10.6
- net GHS3_MOS: now reaches Q3.4, R15.2
- net GHS3_MOS: now also D4.2 (A)
- net CAN_SHDN renamed SEC_IN
- net SEC_IN: now also D208.2 (A), R206.2, R207.1
- new net: Q203.E, R210.2
- new net: Q203.C, R207.2, TP14.1, TP15.1
- new net: Q202.5, Q202.6, Q202.7, Q202.8, R205.1, R211.2
- new net: D206.1 (K), R209.1
- new net: D206.2 (A), Q203.B, R208.2
- new net: D208.1 (K), R212.1
- new net: D207.1 (K), R211.1
- new net GNDPWR: C13.1, C14.1, C15.1, C31.2, C32.2, D202.2 (A), D205.2 (A), NT1.2, Q202.1, Q202.2, Q202.3, R201.1, R204.1, R205.2, R31.2, R32.2, R33.2, R34.2, R35.2, R36.2, R50.1, R51.1, R52.1, TP3.1, TP4.1
Other:
- note added: "NM"
- note added: "R5, R8, R12, R14"
- note added: "VM - 48V VCC - Gate driving supply voltage - 12V VREGIN - 3.3 V LDO linear regulator input - 12V VDD - 3,3V VBAT VDDA VREF+ - 3,3V do dzielnika napiecia GND"
- note removed: "VM - 48V VCC - Gate driving supply voltage - 12V VREGIN - 3.3 V LDO linear regulator input - 12V VDD - 3,3V VBAT VDDA VREF+ GND"
- moved on the sheet: C31, C32, J10

Commit message: add gripper and so on
Parts:
- J10, J9: footprint footprints:M207810345 -> UNIVERSAL_JOINT:M207810345
- R201: value 200 -> 4.5k
- R39: value 72.3k 1% -> 3.01k 1%
- SW3: value SW_MEC_5E -> SKHUALE010
- TP11, TP12, TP13: value TestPoint -> 1-726388-2
Other:
- note added: "A,B DODAĆ RC FILTER 1k 10pF"
- note added: "CONNECTORS"
- note added: "DODAĆ LED ZASILANIA 12V"
- note added: "MOŻNA ZWOLNIĆ"
- note added: "R201 ZAMIENIĆ NA 2 SZTUKI RES SMD 4.7K OHM 5% 1/2W 0805"
- note added: "ZAMIENIĆ NA DRABINKĘ"
- note added: "ZAMIENIĆ NA NETTIE"
- note added: "ZAMIENIĆ UKŁAD HAMULCA NA TRANSIL ???"
- note removed: "CS MA730 - MGH MA730 - MGL MA730 CS MA310 - MGH MA310 - MGL MA310 EMERGENCY OUT EMERGNCY IN BRAKE ENABLED IN DIP1 - DIP2 - DIP3 - DIP4"
- moved on the sheet: C10, C11, C12, C19, C201, C40, C6, C7, C8, C9, D8, J10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

Commit message: update 3.1
Parts:
- TP10, TP14, TP15, TP16, TP17, TP5, TP6, TP7, TP8, TP9: footprint footprints:Pin_D1.2mm_L10.2mm_W2.9mm_FlatFork -> UNIVERSAL_JOINT:61-2348-11_0030
- X1: value Crystal_GND24_Small -> ECS-240-8-36B2-CKM-TR
Other:
- note added: "NOT MOUNTED"
Changed lines of the file:
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@@
     (stroke (width 0) (type default) (color 0 0 0 0))
   )
+  (polyline (pts (xy 820.42 -2.54) (xy 820.42 90.17))
+    (stroke (width 0) (type default) (color 0 0 0 0))
+  )
+  (polyline (pts (xy 820.42 -2.54) (xy 901.7 -2.54))
+    (stroke (width 0) (type default) (color 0 0 0 0))
+  )
+  (polyline (pts (xy 901.7 -2.54) (xy 901.7 90.17))
+    (stroke (width 0) (type default) (color 0 0 0 0))
+  )
+  (polyline (pts (xy 901.7 90.17) (xy 820.42 90.17))
+    (stroke (width 0) (type default) (color 0 0 0 0))
+  )
   (text "VM - 48V\nVCC - Gate driving supply voltage - 12V\nVREGIN - 3.3 V LDO linear regulator input - 12V\nVDD - 3,3V\nVBAT\nVDDA\nVREF+ - 3,3V do dzielnika napiecia\nGND"
     (at 31.75 73.66 0)
@@
     (effects (font (size 1.27 1.27)) (justify left bottom))
   )
+  (text "NOT MOUNTED" (at 821.69 3.81 0)
+    (effects (font (size 3 3)) (justify left bottom))
+  )
   (text "ZAMIENIĆ UKŁAD HAMULCA \nNA TRANSIL ???" (at 826.77 46.99 0)
     (effects (font (size 1.27 1.27)) (justify left bottom))
@@
       (effects (font (size 1.27 1.27)) (justify left))
     )
-    (property "Footprint" "footprints:Pin_D1.2mm_L10.2mm_W2.9mm_FlatFork" (id 2) (at 504.825 247.65 0)
+    (property "Footprint" "UNIVERSAL_JOINT:61-2348-11_0030" (id 2) (at 504.825 247.65 0)
       (effects (font (size 1.27 1.27)) hide)
     )
@@
       (effects (font (size 1.27 1.27)) (justify left))
     )
-    (property "Footprint" "footprints:Pin_D1.2mm_L10.2mm_W2.9mm_FlatFork" (id 2) (at 510.54 247.65 0)
+    (property "Footprint" "UNIVERSAL_JOINT:61-2348-11_0030" (id 2) (at 510.54 247.65 0)
       (effects (font (size 1.27 1.27)) hide)
     )
@@
       (effects (font (size 1.27 1.27)) (justify left))
     )
-    (property "Footprint" "footprints:Pin_D1.2mm_L10.2mm_W2.9mm_FlatFork" (id 2) (at 520.7 247.65 0)
+    (property "Footprint" "UNIVERSAL_JOINT:61-2348-11_0030" (id 2) (at 520.7 247.65 0)
       (effects (font (size 1.27 1.27)) hide)
     )
@@
       (effects (font (size 1.27 1.27)) (justify left))
     )
-    (property "Footprint" "footprints:Pin_D1.2mm_L10.2mm_W2.9mm_FlatFork" (id 2) (at 527.05 247.65 0)
+    (property "Footprint" "UNIVERSAL_JOINT:61-2348-11_0030" (id 2) (at 527.05 247.65 0)
       (effects (font (size 1.27 1.27)) hide)
     )
@@
       (effects (font (size 1.27 1.27)) (justify left))
     )
-    (property "Footprint" "footprints:Pin_D1.2mm_L10.2mm_W2.9mm_FlatFork" (id 2) (at 638.175 74.295 0)
+    (property "Footprint" "UNIVERSAL_JOINT:61-2348-11_0030" (id 2) (at 638.175 74.295 0)
       (effects (font (size 1.27 1.27)) hide)
     )
@@
       (effects (font (size 1.27 1.27)) (justify left))
     )
-    (property "Footprint" "footprints:Pin_D1.2mm_L10.2mm_W2.9mm_FlatFork" (id 2) (at 643.255 74.295 0)
+    (property "Footprint" "UNIVERSAL_JOINT:61-2348-11_0030" (id 2) (at 643.255 74.295 0)
       (effects (font (size 1.27 1.27)) hide)
     )
@@
       (effects (font (size 1.27 1.27)) (justify left))
     )
-    (property "Footprint" "footprints:Pin_D1.2mm_L10.2mm_W2.9mm_FlatFork" (id 2) (at 676.275 74.93 0)
+    (property "Footprint" "UNIVERSAL_JOINT:61-2348-11_0030" (id 2) (at 676.275 74.93 0)
       (effects (font (size 1.27 1.27)) hide)
     )
@@
       (effects (font (size 1.27 1.27)) (justify left))
     )
-    (property "Footprint" "footprints:Pin_D1.2mm_L10.2mm_W2.9mm_FlatFork" (id 2) (at 684.53 74.93 0)
+    (property "Footprint" "UNIVERSAL_JOINT:61-2348-11_0030" (id 2) (at 684.53 74.93 0)
       (effects (font (size 1.27 1.27)) hide)
     )
@@
       (effects (font (size 1.27 1.27)) (justify left))
     )
-    (property "Footprint" "footprints:Pin_D1.2mm_L10.2mm_W2.9mm_FlatFork" (id 2) (at 996.95 24.765 0)
+    (property "Footprint" "UNIVERSAL_JOINT:61-2348-11_0030" (id 2) (at 996.95 24.765 0)
       (effects (font (size 1.27 1.27)) hide)
     )
@@
       (effects (font (size 1.27 1.27)) (justify left))
     )
-    (property "Footprint" "footprints:Pin_D1.2mm_L10.2mm_W2.9mm_FlatFork" (id 2) (at 1003.3 24.765 0)
+    (property "Footprint" "UNIVERSAL_JOINT:61-2348-11_0030" (id 2) (at 1003.3 24.765 0)
       (effects (font (size 1.27 1.27)) hide)
     )
@@
       (effects (font (size 1.27 1.27)) (justify left))
     )
-    (property "Value" "Crystal_GND24_Small" (id 1) (at 295.6561 113.6266 0)
+    (property "Value" "ECS-240-8-36B2-CKM-TR" (id 1) (at 290.5761 114.8966 0)
       (effects (font (size 1.27 1.27)) (justify left))
     )
@@
     )
     (path "/5fbf8a62-a3ce-476c-bcd3-d79f02c7147c"
-      (reference "TP5") (unit 1) (value "12V") (footprint "footprints:Pin_D1.2mm_L10.2mm_W2.9mm_FlatFork")
+      (reference "TP5") (unit 1) (value "12V") (footprint "UNIVERSAL_JOINT:61-2348-11_0030")
     )
     (path "/cd38165a-8748-4408-819a-f5fffe18a24d"
-      (reference "TP6") (unit 1) (value "12V") (footprint "footprints:Pin_D1.2mm_L10.2mm_W2.9mm_FlatFork")
+      (reference "TP6") (unit 1) (value "12V") (footprint "UNIVERSAL_JOINT:61-2348-11_0030")
     )
     (path "/7c29edd1-d98d-42e2-8e0e-eba6b02116ee"
-      (reference "TP7") (unit 1) (value "CANL") (footprint "footprints:Pin_D1.2mm_L10.2mm_W2.9mm_FlatFork")
+      (reference "TP7") (unit 1) (value "CANL") (footprint "UNIVERSAL_JOINT:61-2348-11_0030")
     )
     (path "/af7b0621-f73b-493f-bb0f-1a9cdf257983"
-      (reference "TP8") (unit 1) (value "CANL") (footprint "footprints:Pin_D1.2mm_L10.2mm_W2.9mm_FlatFork")
+      (reference "TP8") (unit 1) (value "CANL") (footprint "UNIVERSAL_JOINT:61-2348-11_0030")
     )
     (path "/e7827ade-328d-4a0e-8a98-f49c35a0b6f4"
-      (reference "TP9") (unit 1) (value "CANH") (footprint "footprints:Pin_D1.2mm_L10.2mm_W2.9mm_FlatFork")
+      (reference "TP9") (unit 1) (value "CANH") (footprint "UNIVERSAL_JOINT:61-2348-11_0030")
     )
     (path "/4c803cfa-b129-45fc-b441-042bcf6c2bb1"
-      (reference "TP10") (unit 1) (value "CANH") (footprint "footprints:Pin_D1.2mm_L10.2mm_W2.9mm_FlatFork")
+      (reference "TP10") (unit 1) (value "CANH") (footprint "UNIVERSAL_JOINT:61-2348-11_0030")
     )
     (path "/fe011b94-1f9b-4ca1-af47-38d9ea9dd2b1"
@@
     )
     (path "/56e89cc4-a6b2-4a21-99ca-470d037adf2d"
-      (reference "TP14") (unit 1) (value "TestPoint") (footprint "footprints:Pin_D1.2mm_L10.2mm_W2.9mm_FlatFork")
+      (reference "TP14") (unit 1) (value "TestPoint") (footprint "UNIVERSAL_JOINT:61-2348-11_0030")
     )
     (path "/16ebd710-a9fa-4ae3-ae30-a4a2ea001b7c"
-      (reference "TP15") (unit 1) (value "TestPoint") (footprint "footprints:Pin_D1.2mm_L10.2mm_W2.9mm_FlatFork")
+      (reference "TP15") (unit 1) (value "TestPoint") (footprint "UNIVERSAL_JOINT:61-2348-11_0030")
     )
     (path "/fe6a0cf8-4610-4fa5-bfda-fd05d3060b60"
-      (reference "TP16") (unit 1) (value "GND") (footprint "footprints:Pin_D1.2mm_L10.2mm_W2.9mm_FlatFork")
+      (reference "TP16") (unit 1) (value "GND") (footprint "UNIVERSAL_JOINT:61-2348-11_0030")
     )
     (path "/53c36bf6-c9ab-410f-a4b6-5581fae06949"
-      (reference "TP17") (unit 1) (value "GND") (footprint "footprints:Pin_D1.2mm_L10.2mm_W2.9mm_FlatFork")
+      (reference "TP17") (unit 1) (value "GND") (footprint "UNIVERSAL_JOINT:61-2348-11_0030")
     )
     (path "/77feccfa-257b-468c-a0fb-d6a724f46f1c"
@@
     )
     (path "/9124cc41-d0bb-4ac4-9425-1f1324ea8733"
-      (reference "X1") (unit 1) (value "Crystal_GND24_Small") (footprint "Crystal:Crystal_SMD_2520-4Pin_2.5x2.0mm")
+      (reference "X1") (unit 1) (value "ECS-240-8-36B2-CKM-TR") (footprint "Crystal:Crystal_SMD_2520-4Pin_2.5x2.0mm")
     )
   )

Commit message: update NM parts
Parts:
- D203: value MBRD20 -> BRIDGED
- D204: value STPS0560Z -> NM
- D205: value ACZRW5242B-G -> NM
- D206: value RED -> NM
- D207: value ORANGE -> NM
- D208: value GREEN -> NM
- Q201: value BC856BWT1G -> NM
- Q202: value IAUC120N06S5L -> NM
- R202: value 10k -> NM
- R203, R204: value 200 -> NM
- R205: value 47R -> NM
- R209: value 130R -> NM
- R211: value 4.6k -> NM
- R212: value 80R -> NM
Other:
- note removed: "ZAMIENIĆ UKŁAD HAMULCA NA TRANSIL ???"

Commit message: MASTER UPDATE
Other:
- note added: "C2 przed rezystorem"
- note added: "DODAĆ FILTR RC DO AB"
- note added: "PRZY SCREF DODAĆ DZIELNIK - BRAK!"
- note added: "ZAMIENIĆ NA DRABINKĘ LUB WYWALIĆ"
- note removed: "ZAMIENIĆ NA DRABINKĘ"
Changed lines of the file:
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@@
     (effects (font (size 3 3)) (justify left bottom))
   )
-  (text "DODAĆ LED ZASILANIA 12V" (at 205.74 188.595 0)
-    (effects (font (size 1.27 1.27)) (justify left bottom))
-  )
-  (text "ZAMIENIĆ NA NETTIE" (at 227.33 173.99 180)
-    (effects (font (size 1.27 1.27)) (justify right bottom))
+  (text "DODAĆ LED ZASILANIA 12V" (at 185.42 187.96 0)
+    (effects (font (size 5 5)) (justify left bottom))
   )
   (text "ZAMIENIĆ NA NETTIE" (at 228.6 198.12 180)
@@
     (effects (font (size 1.27 1.27)) (justify right bottom))
   )
+  (text "ZAMIENIĆ NA NETTIE" (at 267.335 163.195 180)
+    (effects (font (size 5 5)) (justify right bottom))
+  )
   (text "A,B DODAĆ RC FILTER\n1k 10pF" (at 333.375 215.9 0)
     (effects (font (size 1.27 1.27)) (justify left bottom))
+  )
+  (text "PRZY SCREF DODAĆ DZIELNIK - BRAK!" (at 334.01 232.41 0)
+    (effects (font (size 5 5)) (justify left bottom))
   )
   (text "MOŻNA ZWOLNIĆ" (at 336.55 208.28 0)
@@
     (effects (font (size 1.27 1.27)) (justify left bottom))
   )
-  (text "ZAMIENIĆ NA DRABINKĘ" (at 442.595 123.19 0)
-    (effects (font (size 1.27 1.27)) (justify left bottom))
+  (text "DODAĆ FILTR RC DO AB" (at 342.265 223.52 0)
+    (effects (font (size 5 5)) (justify left bottom))
+  )
+  (text "C2 przed rezystorem" (at 345.44 217.805 0)
+    (effects (font (size 5 5)) (justify left bottom))
+  )
+  (text "ZAMIENIĆ NA DRABINKĘ LUB WYWALIĆ" (at 440.055 126.365 0)
+    (effects (font (size 5 5)) (justify left bottom))
   )
   (text "R5, R8, R12, R14" (at 443.23 145.415 270)
@@
     (effects (font (size 1.27 1.27) (thickness 0.254) bold) (justify left bottom))
   )
-  (text "NM" (at 680.72 160.02 0)
-    (effects (font (size 1.27 1.27) (thickness 0.254) bold) (justify left bottom))
-  )

Commit message: update to newest
Other:
- moved on the sheet: C1, C10, C11, C12, C13, C14, C15, C16, C17, C18, C19, C2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
