File: GRIPPER_TWO_ADVANCED_CONECTION_BOARD_v1.2/GRIPPER_TWO_ADVANCED_CONECTION_BOARD.kicad_pcb (KiCad board)
At the start: 2 copper layers, 44.5 x 95.1 mm, 29 parts, among them J1 Conn_01x02_Male

Commit message: udpate
Parts:
- added R1: 100, footprints:R_0603_1608Metric_Pad0.98x0.95mm_HandSolder, F.Cu at (170.4, 146.3)
- added R2: 100, footprints:R_0603_1608Metric_Pad0.98x0.95mm_HandSolder, F.Cu at (167.9, 146.3)
- added R3: 100, footprints:R_0603_1608Metric_Pad0.98x0.95mm_HandSolder, F.Cu at (150.0, 152.5)
- J1: value Conn_01x02_Male -> Conn_01x03_Male; footprint footprints:PinHeader_1x02_P2.54mm_Vertical -> footprints:PinHeader_1x03_P2.54mm_Vertical
- moved J1 3.11 mm to (170.4, 151.9)
- moved TP2 0.90 mm to (162.9, 149.0)
- moved TP4 0.90 mm to (159.7, 149.0)
- moved TP5 0.90 mm to (158.1, 149.0)
- moved TP6 0.90 mm to (156.5, 149.0)
- moved TP7 0.90 mm to (154.9, 149.0)
- moved TP1 0.90 mm to (153.3, 149.0)
- moved TP3 0.90 mm to (161.3, 149.0)
Connections:
- J1 pad 1: /RX -> Net-(J1-Pad1)
- J1 pad 2: /TX -> Net-(J1-Pad2)
Routing:
- net /GND: track 94.0 -> 112.0 mm
- net GNDPWR: track 103.1 -> 111.2 mm
- net /CAN+: track 94.7 -> 99.8 mm
- net Net-(J1-Pad2): track 0.00 -> 4.70 mm
- net Net-(J1-Pad1): track 0.00 -> 4.69 mm
- net /TX: track 96.2 -> 92.1 mm
- net /RX: track 96.6 -> 92.5 mm
- net /SAFETY: track 96.5 -> 95.7 mm
- net /CAN-: track 99.4 -> 100.0 mm
Other:
- board text added: "POLA LUTOWNICZE CO 1,28 mm pola wyzsze do 3mm"
- board text removed: "POLA LUTOWNICZE CO 1,64mm"
