File: GRIPPER_TWO_ADVANCED_CONECTION_BOARD_v1.2/GRIPPER_TWO_ADVANCED_CONECTION_BOARD.kicad_sch (KiCad schematic)
At the start: 29 parts, among them J1 Conn_01x02_Male

Commit message: udpate
Parts:
- added R1, R2, R3: 100, footprints:R_0603_1608Metric_Pad0.98x0.95mm_HandSolder, symbol Device:R_Small
- J1: value Conn_01x02_Male -> Conn_01x03_Male; footprint footprints:PinHeader_1x02_P2.54mm_Vertical -> footprints:PinHeader_1x03_P2.54mm_Vertical; symbol Connector:Conn_01x02_Male -> Connector:Conn_01x03_Male
Connections:
- net GND: now also J1.3 (Pin_3), R3.2
- net GNDPWR: now also R3.1
- net RX: now also R1.2; no longer J1.1 (Pin_1)
- net TX: now also R2.2; no longer J1.2 (Pin_2)
- new net: J1.2 (Pin_2), R2.1
- new net: J1.1 (Pin_1), R1.1
Changed lines of the file:
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@@
+    (stroke (width 0) (type default) (color 0 0 0 0))
+  )
+  (wire (pts (xy 50.165 121.285) (xy 55.245 121.285))
     (stroke (width 0) (type default) (color 0 0 0 0))
   )
@@
     (stroke (width 0) (type default) (color 0 0 0 0))
   )
+  (wire (pts (xy 187.96 71.755) (xy 174.625 71.755))
+    (stroke (width 0) (type default) (color 0 0 0 0))
+  )
+  (wire (pts (xy 60.325 121.285) (xy 66.675 121.285))
+    (stroke (width 0) (type default) (color 0 0 0 0))
+  )
   (wire (pts (xy 142.24 106.68) (xy 190.5 106.68))
     (stroke (width 0) (type default) (color 0 0 0 0))
@@
     (stroke (width 0) (type default) (color 0 0 0 0))
   )
+  (wire (pts (xy 178.435 69.215) (xy 174.625 69.215))
+    (stroke (width 0) (type default) (color 0 0 0 0))
+  )
   (wire (pts (xy 44.45 89.535) (xy 44.45 92.075))
     (stroke (width 0) (type default) (color 0 0 0 0))
@@
     (stroke (width 0) (type default) (color 0 0 0 0))
   )
+  (wire (pts (xy 187.96 69.215) (xy 183.515 69.215))
+    (stroke (width 0) (type default) (color 0 0 0 0))
+  )
   (wire (pts (xy 44.45 67.31) (xy 44.45 69.85))
     (stroke (width 0) (type default) (color 0 0 0 0))
@@
     (stroke (width 0) (type default) (color 0 0 0 0))
   )
+  (wire (pts (xy 187.96 66.675) (xy 183.515 66.675))
+    (stroke (width 0) (type default) (color 0 0 0 0))
+  )
   (wire (pts (xy 44.45 36.83) (xy 64.77 36.83))
     (stroke (width 0) (type default) (color 0 0 0 0))
   )
+  (wire (pts (xy 178.435 66.675) (xy 174.625 66.675))
+    (stroke (width 0) (type default) (color 0 0 0 0))
+  )
   (wire (pts (xy 44.45 83.82) (xy 44.45 86.36))
     (stroke (width 0) (type default) (color 0 0 0 0))
@@
     (effects (font (size 1.27 1.27)) (justify left bottom))
   )
-  (label "RX" (at 174.625 69.215 0)
+  (label "RX" (at 187.96 66.675 0)
     (effects (font (size 1.27 1.27)) (justify left bottom))
   )
@@
     (effects (font (size 1.27 1.27)) (justify left bottom))
   )
-  (label "TX" (at 174.625 71.755 0)
+  (label "TX" (at 187.96 69.215 0)
     (effects (font (size 1.27 1.27)) (justify left bottom))
   )
@@
   )
   (label "CAN+" (at 52.07 43.18 0)
+    (effects (font (size 1.27 1.27)) (justify left bottom))
+  )
+  (label "GND" (at 66.675 121.285 0)
     (effects (font (size 1.27 1.27)) (justify left bottom))
   )
@@
     (effects (font (size 1.27 1.27)) (justify left bottom))
   )
+  (label "GND" (at 187.96 71.755 0)
+    (effects (font (size 1.27 1.27)) (justify left bottom))
+  )
   (label "RX" (at 64.77 97.79 0)
     (effects (font (size 1.27 1.27)) (justify left bottom))
@@
     (effects (font (size 1.27 1.27)) (justify left bottom))
   )
+  (label "GNDPWR" (at 50.165 121.285 180)
+    (effects (font (size 1.27 1.27)) (justify right bottom))
+  )
   (symbol (lib_id "power:GNDPWR") (at 152.4 111.76 0) (unit 1)
     (in_bom yes) (on_board yes) (fields_autoplaced)
@@
     (pin "1")
   )
+  (symbol (lib_id "Device:R_Small") (at 57.785 121.285 90) (unit 1)
+    (in_bom yes) (on_board yes)
+    (property "Reference" "R3" (id 0) (at 54.61 120.015 90))
+    (property "Value" "100" (id 1) (at 61.595 120.015 90))
+    (property "Footprint" "footprints:R_0603_1608Metric_Pad0.98x0.95mm_HandSolder" (id 2) (at 57.785 121.285 0)
+      (effects (font (size 1.27 1.27)) hide)
+    )
+    (property "Datasheet" "~" (id 3) (at 57.785 121.285 0)
+      (effects (font (size 1.27 1.27)) hide)
+    )
+    (pin "1")
+    (pin "2")
+  )
   (symbol (lib_name "SMD2_4") (lib_id "Gripper Connection Board-eagle-import:SMD2") (at 41.91 80.645 0) (unit 1)
     (in_bom yes) (on_board yes)
@@
     (pin "1")
   )
+  (symbol (lib_id "Device:R_Small") (at 180.975 69.215 90) (unit 1)
+    (in_bom yes) (on_board yes)
+    (property "Reference" "R2" (id 0) (at 177.8 70.485 90))
+    (property "Value" "100" (id 1) (at 184.785 70.485 90))
+    (property "Footprint" "footprints:R_0603_1608Metric_Pad0.98x0.95mm_HandSolder" (id 2) (at 180.975 69.215 0)
+      (effects (font (size 1.27 1.27)) hide)
+    )
+    (property "Datasheet" "~" (id 3) (at 180.975 69.215 0)
+      (effects (font (size 1.27 1.27)) hide)
+    )
+    (pin "1")
+    (pin "2")
+  )
   (symbol (lib_id "Gripper Connection Board-eagle-import:SE11") (at 193.04 127 270) (unit 1)
     (in_bom yes) (on_board yes)
@@
     (pin "MP")
   )
-  (symbol (lib_id "Connector:Conn_01x02_Male") (at 169.545 69.215 0) (unit 1)
-    (in_bom yes) (on_board yes) (fields_autoplaced)
+  (symbol (lib_id "Connector:Conn_01x03_Male") (at 169.545 69.215 0) (unit 1)
+    (in_bom yes) (on_board yes)
     (property "Reference" "J1" (id 0) (at 172.0469 63.5 0))
-    (property "Value" "Conn_01x02_Male" (id 1) (at 172.0469 66.04 0))
-    (property "Footprint" "footprints:PinHeader_1x02_P2.54mm_Vertical" (id 2) (at 169.545 69.215 0)
+    (property "Value" "Conn_01x03_Male" (id 1) (at 167.64 69.215 90))
+    (property "Footprint" "footprints:PinHeader_1x03_P2.54mm_Vertical" (id 2) (at 169.545 69.215 0)
       (effects (font (size 1.27 1.27)) hide)
     )
@@
     (pin "1")
     (pin "2")
+    (pin "3")
   )
   (symbol (lib_id "Gripper Connection Board-eagle-import:SE11") (at 193.04 124.46 270) (unit 1)
@@
     )
     (property "Datasheet" "" (id 3) (at 41.91 97.79 0)
+      (effects (font (size 1.27 1.27)) hide)
+    )
+    (pin "1")
+    (pin "2")
+  )
+  (symbol (lib_id "Device:R_Small") (at 180.975 66.675 90) (unit 1)
+    (in_bom yes) (on_board yes)
+    (property "Reference" "R1" (id 0) (at 177.8 65.405 90))
+    (property "Value" "100" (id 1) (at 184.785 65.405 90))
+    (property "Footprint" "footprints:R_0603_1608Metric_Pad0.98x0.95mm_HandSolder" (id 2) (at 180.975 66.675 0)
+      (effects (font (size 1.27 1.27)) hide)
+    )
+    (property "Datasheet" "~" (id 3) (at 180.975 66.675 0)
       (effects (font (size 1.27 1.27)) hide)
     )
@@
     )
     (path "/1d2ec7fc-c8bc-422f-a55c-dc298087d605"
-      (reference "J1") (unit 1) (value "Conn_01x02_Male") (footprint "footprints:PinHeader_1x02_P2.54mm_Vertical")
+      (reference "J1") (unit 1) (value "Conn_01x03_Male") (footprint "footprints:PinHeader_1x03_P2.54mm_Vertical")
     )
     (path "/31d508ce-d492-43bc-8596-57364a32a27b"
@@
       (reference "PGND1") (unit 1) (value "SMD2") (footprint "Gripper Connection Board:SMD1,27-2,54")
     )
+    (path "/c121c6a8-bf2a-4d06-bdfc-3870baa058dc"
+      (reference "R1") (unit 1) (value "100") (footprint "footprints:R_0603_1608Metric_Pad0.98x0.95mm_HandSolder")
+    )
+    (path "/15d33ba9-67a6-4431-8cba-40cb1f099b0e"
+      (reference "R2") (unit 1) (value "100") (footprint "footprints:R_0603_1608Metric_Pad0.98x0.95mm_HandSolder")
+    )
+    (path "/03905ff5-df18-48aa-8be8-13440887926d"
+      (reference "R3") (unit 1) (value "100") (footprint "footprints:R_0603_1608Metric_Pad0.98x0.95mm_HandSolder")
+    )
     (path "/db4bfdba-1a01-4b47-a87b-0a55fd70c815"
