File: GRIPPER_TWO_ADVANCED_CONTROL_BOARD_v1.2/GRIPPER_TWO_ADVANCED_CONTROL_BOARD_v1_2.kicad_sch (KiCad schematic)
At the start: 70 parts, among them IC1 BD9G341AEFJ-E2, J1 Conn_01x04_Male, J2 59453-061110ECHLF, J3 59453-061110ECHLF, Q1 NPN-TRANSISTOR_SOT23, Q2 2PC4081S,115, Q3 SQ7415EN, U1 STM32G431KBT6, U2 STR485LVQT, U3 INA282AID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

Commit message: udpate
Other:
- moved on the sheet: C1, C10, C11, C12, C13, C14, C15, C2, C6, C7, D3, D4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
