File: GRIPPER_TWO_ADVANCED_CONTROL_BOARD_v1.3/GRIPPER_TWO_ADVANCED_CONTROL_BOARD_v1_3.kicad_pcb (KiCad board)
At the start: 2 copper layers, 46 x 39 mm, 72 parts, among them IC1 BD9G341AEFJ-E2, J1 Conn_01x04_Male, J2 59453-061110ECHLF, J3 59453-061110ECHLF, Q1 NPN-TRANSISTOR_SOT23, Q2 2PC4081S,115, Q3 SQ7415EN, U1 STM32G431KBT6, U2 STR485LVQT, U3 INA282AID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

Commit message: udpate
Parts:
- removed D2: RED, footprints:D_0603_1608Metric_Pad1.05x0.95mm_HandSolder
- removed NT1: NetTie_2, footprints:NetTie-2_SMD_Pad0.5mm
- added LED1: RED, footprints:D_0603_1608Metric_Pad1.05x0.95mm_HandSolder, F.Cu at (179.3, 85.8)
- added LED2: GREEN, footprints:D_0603_1608Metric_Pad1.05x0.95mm_HandSolder, F.Cu at (177.6, 85.8)
- added Q4: BSS138, footprints:SOT-23, F.Cu at (173.6, 85.9)
- added R31: 10k, footprints:R_0603_1608Metric_Pad0.98x0.95mm_HandSolder, F.Cu at (177.8, 91.0)
- added R32: 1,1k, footprints:R_0603_1608Metric_Pad0.98x0.95mm_HandSolder, F.Cu at (175.0, 91.1)
- added R33: 100, footprints:R_0603_1608Metric_Pad0.98x0.95mm_HandSolder, F.Cu at (177.8, 94.3)
- added TP1: TestPoint, footprints:TestPoint_Pad_1.0x1.0mm, F.Cu at (150.1, 105.2)
- added TP2: TestPoint, footprints:TestPoint_Pad_1.0x1.0mm, F.Cu at (150.1, 107.2)
- D1: value GREEN -> BAT30K
- Q2: value 2PC4081S,115 -> BSS138; footprint GRIPPER_TWO_ADVANCED_CONTROL_BOARD:SOT23-EBC -> footprints:SOT-23
- R16: value 5,23k -> 1,5k
- R17: value 487 -> 1k
- R18: value 13,7k -> 1k
- R19, R21: value 200R -> 10k
- R20: value 60 -> 100
- moved Q2 10.7 mm to (169.7, 85.9), turned to 0 degrees
- moved R21 9.00 mm to (173.9, 88.4), turned to 0 degrees
- moved R20 8.84 mm to (170.5, 88.4), turned to 0 degrees
- moved D1 8.68 mm to (175.0, 94.4), turned to -90 degrees
- moved R18 4.36 mm to (180.8, 94.3), turned to 90 degrees
- moved R17 3.34 mm to (173.3, 91.0), turned to 90 degrees
- moved C13 3.04 mm to (156.4, 86.0), turned to 90 degrees
- moved D7 2.80 mm to (163.0, 86.4)
- moved R19 2.79 mm to (180.8, 91.0), turned to 90 degrees
- moved R16 1.60 mm to (179.3, 89.2)
- moved J2 1.60 mm to (151.7, 102.4)
- moved R26 1.27 mm to (154.9, 86.0), turned to 90 degrees
- moved C17 0.20 mm to (169.6, 91.0)
Connections:
- net /24V renamed +24V
- D1 pad 2: /SEC -> /SAFETY
- R16 pad 1: GND -> Net-(LED1-Pad1)
- R16 pad 2: /SEC_IN -> GND
- R17 pad 1: Net-(D1-Pad1) -> +12V
- R17 pad 2: GND -> /SAFETY
- R18 pad 1: /SEC_IN -> /SEC_OUT
- R18 pad 2: /SEC -> Net-(Q2-Pad1)
- R19 pad 1: /SEC_OUT -> Net-(Q2-Pad1)
- R19 pad 2: Net-(Q2-PadB) -> GND
- R20 pad 1: Net-(D2-Pad1) -> Net-(D1-Pad1)
- R20 pad 2: GND -> Net-(Q4-Pad1)
- R21 pad 1: GND -> Net-(Q4-Pad1)
- R21 pad 2: Net-(Q2-PadE) -> GND
Routing:
- net /SEC: track 39.6 -> 0.00 mm, vias 2 -> 0
- net /SAFETY: track 0.00 -> 33.5 mm, vias 0 -> 2
- net +3V3: track 154.8 -> 179.3 mm, vias 11 -> 13
- net Net-(Q2-Pad1): track 0.00 -> 17.0 mm, vias 0 -> 2
- net Net-(Q4-Pad3): track 0.00 -> 14.7 mm
- net Net-(D1-Pad1): track 1.61 -> 11.0 mm, vias 0 -> 2
- net /SEC_IN: track 30.5 -> 24.2 mm
- net Net-(LED2-Pad1): track 0.00 -> 4.62 mm
- net +12V: track 41.5 -> 45.3 mm
- net /SPI_CLK: track 50.5 -> 54.3 mm
- net Net-(Q4-Pad1): track 0.00 -> 3.77 mm
- net Net-(C13-Pad1): track 7.60 -> 10.8 mm
- net /SPI_MOSI: track 53.8 -> 55.5 mm
- net Net-(Q2-PadE): track 1.65 -> 0.00 mm
- net Net-(Q2-PadB): track 1.65 -> 0.00 mm
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