File: GRIPPER_TWO_ADVANCED_CONTROL_BOARD_v1.3/GRIPPER_TWO_ADVANCED_CONTROL_BOARD_v1_3.kicad_sch (KiCad schematic)
At the start: 86 parts, among them IC1 BD9G341AEFJ-E2, J1 Conn_01x04_Male, J2 59453-061110ECHLF, J3 59453-061110ECHLF, Q1 NPN-TRANSISTOR_SOT23, Q2 2PC4081S,115, Q3 SQ7415EN, U1 STM32G431KBT6, U2 STR485LVQT, U3 INA282AID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

Commit message: udpate
Parts:
- removed D1: GREEN, footprints:D_0603_1608Metric_Pad1.05x0.95mm_HandSolder, symbol Device:LED
- removed D2: RED, footprints:D_0603_1608Metric_Pad1.05x0.95mm_HandSolder, symbol Device:LED
- removed NT1: NetTie_2, footprints:NetTie-2_SMD_Pad0.5mm, symbol Device:NetTie_2
- removed Q2: 2PC4081S,115, GRIPPER_TWO_ADVANCED_CONTROL_BOARD:SOT23-EBC, symbol UNIVERSAL_JOINT_v2_1-eagle-import:-NPN-SOT23-EBC
- removed R16: 5,23k, footprints:R_0603_1608Metric_Pad0.98x0.95mm_HandSolder, symbol Device:R
- removed R17: 487, footprints:R_0603_1608Metric_Pad0.98x0.95mm_HandSolder, symbol Device:R
- removed R18: 13,7k, footprints:R_0603_1608Metric_Pad0.98x0.95mm_HandSolder, symbol Device:R
- removed R19, R21: 200R, footprints:R_0603_1608Metric_Pad0.98x0.95mm_HandSolder, symbol Device:R
- removed R20: 60, footprints:R_0603_1608Metric_Pad0.98x0.95mm_HandSolder, symbol Device:R
- added TP1, TP2: TestPoint, footprints:TestPoint_Pad_1.0x1.0mm, symbol Connector:TestPoint
- gave numbers to parts that had none: 14
Connections:
- net GND: now also TP1.1
- net GNDPWR: now also TP2.1
- net 24V renamed +24V
Other:
- note added: "NM"
