File: UNIVERSAL_HALL_PCB_RI70_v3.0/universal_hall_pcb_RI70_v3.0.kicad_sch (KiCad schematic)
At the start: 9 parts, among them J1 Conn_02x06_Odd_Even, U1 MA710

Commit message: udpate
Parts:
- R1, R2: value 10k -> 10k 1%
Changed lines of the file:
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@@
   )
   (symbol (lib_id "Device:R") (at 213.36 85.09 0) (unit 1)
-    (in_bom yes) (on_board yes) (fields_autoplaced)
-    (property "Reference" "R2" (id 0) (at 215.1381 84.1815 0)
-      (effects (font (size 1.27 1.27)) (justify left))
-    )
-    (property "Value" "10k" (id 1) (at 215.1381 86.9566 0)
+    (in_bom yes) (on_board yes)
+    (property "Reference" "R2" (id 0) (at 215.9 83.8199 0)
+      (effects (font (size 1.27 1.27)) (justify left))
+    )
+    (property "Value" "10k 1%" (id 1) (at 210.82 88.265 90)
       (effects (font (size 1.27 1.27)) (justify left))
     )
@@
   )
   (symbol (lib_id "Device:R") (at 184.785 85.09 0) (unit 1)
-    (in_bom yes) (on_board yes) (fields_autoplaced)
+    (in_bom yes) (on_board yes)
     (property "Reference" "R1" (id 0) (at 186.69 83.8199 0)
       (effects (font (size 1.27 1.27)) (justify left))
     )
-    (property "Value" "10k" (id 1) (at 186.69 86.3599 0)
+    (property "Value" "10k 1%" (id 1) (at 182.245 88.265 90)
       (effects (font (size 1.27 1.27)) (justify left))
     )
@@
     )
     (path "/fdb45f06-8432-4b6f-aa66-6ccbb4707674"
-      (reference "R1") (unit 1) (value "10k") (footprint "footprints:R_0603_1608Metric_Pad0.98x0.95mm_HandSolder")
+      (reference "R1") (unit 1) (value "10k 1%") (footprint "footprints:R_0603_1608Metric_Pad0.98x0.95mm_HandSolder")
     )
     (path "/59db2b12-ce10-4882-91dc-94988ee17a89"
-      (reference "R2") (unit 1) (value "10k") (footprint "footprints:R_0603_1608Metric_Pad0.98x0.95mm_HandSolder")
+      (reference "R2") (unit 1) (value "10k 1%") (footprint "footprints:R_0603_1608Metric_Pad0.98x0.95mm_HandSolder")
     )
     (path "/3869714a-3af0-42a8-92c5-c4f5f72169fd"
