File: UNIVERSAL_JOINT_v2_2/UNIVERSAL_JOINT_v2_2.kicad_pcb (KiCad board)
At the start: 2 copper layers, 76 x 76 mm, 127 parts, among them J1 Conn_02x07_Odd_Even, J10 HEADER_MALE_2X3_2.54_SMT, J9 HEADER_MALE_2X3_2.54_SMT, Q1 NVMFS4C03N, Q2 NVMFS4C03N, Q3 NVMFS4C03N, Q4 NVMFS4C03N, Q5 NVMFS4C03N, Q6 NVMFS4C03N, Q7 BC856BWT1G, Q8 NVMFS4C03N, SW1 SKHMPE010, T1 2PC4081S,115, T2 2PC4081S,115, U1 DRV8323RHRGZR, U2 TCAN332G, U3 STM32G431C8T6, U4 MA730, X1 LFXTAL069392CUTT

Commit message: add gripper and so on
Parts:
- J10: value HEADER_MALE_2X3_2.54_SMT -> n.m.
- Q1, Q2, Q3, Q4, Q5, Q6, Q8: value NVMFS4C03N -> IAUC120N06S5L
- Q7: value BC856BWT1G -> ZXTP19100CFFCT
- U$29: value MBRD20 -> MBRD10100CT
Connections:
- net /HALL_1 renamed /A
- net /HALL_2 renamed /B
Routing:
- net unconnected-(U1-Pad3): track 2.97 -> 0.00 mm
- net unconnected-(C1-Pad2): track 0.00 -> 2.97 mm
- net unconnected-(U1-Pad4): track 2.29 -> 0.00 mm
- net unconnected-(C1-Pad1): track 0.00 -> 2.29 mm

Commit message: UJ 2.2 remove brake resistor
Parts:
- D3, U$1, U$3, U$4: footprint UNIVERSAL_JOINT_v2_2:SMB -> UNIVERSAL_JOINT:SMB
- Q1, Q2, Q3, Q4, Q5, Q6, Q8: footprint UNIVERSAL_JOINT_v2_2:SO-8FL -> UNIVERSAL_JOINT:SO-8FL
- Q7: footprint UNIVERSAL_JOINT_v2_2:SOT23 -> UNIVERSAL_JOINT:SOT23
- SW1: footprint UNIVERSAL_JOINT_v2_2:SKHMPXE010 -> UNIVERSAL_JOINT:SKHMPXE010
- T1, T2: footprint UNIVERSAL_JOINT_v2_2:SOT23-EBC -> UNIVERSAL_JOINT:SOT23-EBC
- U$29: footprint UNIVERSAL_JOINT_v2_2:DPACK -> UNIVERSAL_JOINT:DPACK
- U$6: footprint UNIVERSAL_JOINT_v2_2:BEADC4040X120N -> UNIVERSAL_JOINT:BEADC4040X120N
- U1: footprint UNIVERSAL_JOINT_v2_2:QFN50P700X700X100-49N -> UNIVERSAL_JOINT:QFN50P700X700X100-49N
- U3: footprint UNIVERSAL_JOINT_v2_2:LQFP48-7X7 -> UNIVERSAL_JOINT:LQFP48-7X7
- X1: footprint UNIVERSAL_JOINT_v2_2:2.5X2-4-PAD -> UNIVERSAL_JOINT:2.5X2-4-PAD
Connections:
- net Net-(R23-Pad2) renamed /SECURITY
Routing:
- net unconnected-(U1-Pad4): track 0.00 -> 2.29 mm
- net unconnected-(C1-Pad1): track 2.29 -> 0.00 mm

Commit message: MASTER UPDATE
Parts:
- C1, C10, C11, C12, C18, C19, C2, C20, C21, C22, C23, C24, C25, C3, C36, C38, C39, C5, C6, C7, C8, C9: footprint Capacitor_SMD:C_0603_1608Metric_Pad1.08x0.95mm_HandSolder -> footprints:C_0603_1608Metric_Pad1.08x0.95mm_HandSolder
- C13, C16, C17, C4: footprint Capacitor_SMD:C_0805_2012Metric_Pad1.18x1.45mm_HandSolder -> footprints:C_0805_2012Metric_Pad1.18x1.45mm_HandSolder
- D1, D5, U$10, U$16, U$22, U$23, U$24: footprint Diode_SMD:D_SOD-123 -> footprints:D_SOD-123
- JP1, JP2, JP3, JP4: footprint Jumper:SolderJumper-2_P1.3mm_Open_TrianglePad1.0x1.5mm -> footprints:SolderJumper-2_P1.3mm_Open_TrianglePad1.0x1.5mm
- LED1, LED2, LED3, LED4, LED5, LED6, LED7: footprint Diode_SMD:D_0603_1608Metric_Pad1.05x0.95mm_HandSolder -> footprints:D_0603_1608Metric_Pad1.05x0.95mm_HandSolder
- R1, R10, R11, R12, R13, R14, R15, R16, R17, R18, R19, R2, R20, R22, R23, R25, R26, R27, R28, R30, R31, R36, R37, R5, R51, R54, R55, R56, R58, R6, R7, R8, R9: footprint Resistor_SMD:R_0603_1608Metric_Pad0.98x0.95mm_HandSolder -> footprints:R_0603_1608Metric_Pad0.98x0.95mm_HandSolder
- R21, R3, R4: footprint Resistor_SMD:R_2512_6332Metric_Pad1.40x3.35mm_HandSolder -> footprints:R_2512_6332Metric_Pad1.40x3.35mm_HandSolder
- TP1, TP13, TP14, TP15, TP2, TP3, TP4: footprint Connector_Pin:Pin_D1.3mm_L11.3mm_W2.8mm_Flat -> UNIVERSAL_JOINT:61-2348-11_0030
- TP10, TP11, TP12, TP16, TP17, TP5, TP6, TP7, TP8, TP9: footprint Connector_Pin:Pin_D1.2mm_L11.3mm_W3.0mm_Flat -> UNIVERSAL_JOINT:61-2348-11_0030
Connections:
- C1 pad 1: unconnected-(C1-Pad1) -> Net-(U1-Pad4)
- C1 pad 2: unconnected-(C1-Pad2) -> Net-(U1-Pad3)
- U1 pad 3: unconnected-(U1-Pad3) -> Net-(U1-Pad3)
- U1 pad 4: unconnected-(U1-Pad4) -> Net-(U1-Pad4)
Routing:
- net unconnected-(C1-Pad2): track 2.97 -> 0.00 mm
- net Net-(U1-Pad3): track 0.00 -> 2.97 mm
- net unconnected-(U1-Pad4): track 2.29 -> 0.00 mm
- net Net-(U1-Pad4): track 0.00 -> 2.29 mm

Commit message: udpate
Parts:
- added U5: STM32G431CBU6, UNIVERSAL_JOINT:QFN50P700X700X65-49N-D, F.Cu at (164.1, 119.8)
- moved C20 9.17 mm to (172.3, 115.6), turned to 90 degrees
- moved R20 7.16 mm to (172.3, 118.9), turned to -90 degrees
Connections:
- C25 pad 2: Net-(C25-Pad2) -> +3V3
- U2 pad 3: Net-(C25-Pad2) -> +3V3
Routing:
- net /SWCLK/JTCK: track 10.7 -> 37.1 mm, vias 0 -> 4
- net /JTDI: track 14.7 -> 0.00 mm, vias 2 -> 0
- net /SWDIO/JTMS: track 11.7 -> 0.00 mm, vias 2 -> 0
- net /CS1: track 16.8 -> 7.64 mm
- net +3V3: track 177.1 -> 182.5 mm, vias 13 -> 15
- net /TEMP: track 33.5 -> 38.4 mm
- net /DIP1: track 20.6 -> 25.4 mm
- net /DIP2: track 18.6 -> 23.3 mm
- net /CURR_FB_U: track 49.6 -> 53.8 mm
- net Net-(C24-Pad2): track 47.1 -> 50.0 mm
- net /SPI_MISO: track 18.7 -> 20.4 mm
- net /BRAKE: track 15.2 -> 13.8 mm, vias 2 -> 1
- net Net-(C22-Pad2): track 9.41 -> 8.04 mm
- net /SPI_SCK: track 22.5 -> 23.9 mm
- net /PWM_2: track 38.2 -> 39.4 mm
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Other:
- board text added: "Universal Joint v2.2.B"
- board text removed: "Universal Joint v2.2"
