File: UNIVERSAL_JOINT_v2_2/UNIVERSAL_JOINT_v2_2.kicad_sch (KiCad schematic)
At the start: 128 parts, among them J1 Conn_02x07_Odd_Even, J10 HEADER_MALE_2X3_2.54_SMT, J9 HEADER_MALE_2X3_2.54_SMT, Q1 NVMFS4C03N, Q2 NVMFS4C03N, Q3 NVMFS4C03N, Q4 NVMFS4C03N, Q5 NVMFS4C03N, Q6 NVMFS4C03N, Q7 BC856BWT1G, Q8 NVMFS4C03N, Q9 PZT2222A, SW1 SKHMPE010, T1 2PC4081S,115, T2 2PC4081S,115, U1 DRV8323RHRGZR, U2 TCAN332G, U3 STM32G431C8T6, U4 MA730, X1 LFXTAL069392CUTT

Commit message: add gripper and so on
Parts:
- removed Q9: PZT2222A, Package_TO_SOT_SMD:SOT-223-3_TabPin2, symbol Transistor_BJT:PZT2222A
- J10: value HEADER_MALE_2X3_2.54_SMT -> n.m.
- Q1, Q2, Q3, Q4, Q5, Q6, Q8: value NVMFS4C03N -> IAUC120N06S5L
- Q7: value BC856BWT1G -> ZXTP19100CFFCT
- U$29: value MBRD20 -> MBRD10100CT
Connections:
- net SECURITY: now reaches R23.2, T2.C, TP16.1, TP17.1
- net HALL_1 renamed A
- net HALL_2 renamed B
Other:
- note added: "GATE DRIVER"
- note added: "POWER"
- note added: "SECURITY"
- note added: "uC"
- moved on the sheet: C11, C14, C15, C16, C17, C18, C19, C20, C21, C22, C23, C24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

Commit message: UJ 2.2 remove brake resistor
Parts:
- D3, U$1, U$3, U$4: footprint UNIVERSAL_JOINT_v2_2:SMB -> UNIVERSAL_JOINT:SMB
- Q1, Q2, Q3, Q4, Q5, Q6, Q8: footprint UNIVERSAL_JOINT_v2_2:SO-8FL -> UNIVERSAL_JOINT:SO-8FL
- Q7: footprint UNIVERSAL_JOINT_v2_2:SOT23 -> UNIVERSAL_JOINT:SOT23
- SW1: footprint UNIVERSAL_JOINT_v2_2:SKHMPXE010 -> UNIVERSAL_JOINT:SKHMPXE010
- T1, T2: footprint UNIVERSAL_JOINT_v2_2:SOT23-EBC -> UNIVERSAL_JOINT:SOT23-EBC
- U$29: footprint UNIVERSAL_JOINT_v2_2:DPACK -> UNIVERSAL_JOINT:DPACK
- U$6: footprint UNIVERSAL_JOINT_v2_2:BEADC4040X120N -> UNIVERSAL_JOINT:BEADC4040X120N
- U1: footprint UNIVERSAL_JOINT_v2_2:QFN50P700X700X100-49N -> UNIVERSAL_JOINT:QFN50P700X700X100-49N
- U3: footprint UNIVERSAL_JOINT_v2_2:LQFP48-7X7 -> UNIVERSAL_JOINT:LQFP48-7X7
- X1: footprint UNIVERSAL_JOINT_v2_2:2.5X2-4-PAD -> UNIVERSAL_JOINT:2.5X2-4-PAD

Commit message: MASTER UPDATE
Parts:
- C1, C10, C11, C12, C18, C19, C2, C20, C21, C22, C23, C24, C25, C3, C36, C38, C39, C5, C6, C7, C8, C9: footprint Capacitor_SMD:C_0603_1608Metric_Pad1.08x0.95mm_HandSolder -> footprints:C_0603_1608Metric_Pad1.08x0.95mm_HandSolder
- C13, C16, C17, C4: footprint Capacitor_SMD:C_0805_2012Metric_Pad1.18x1.45mm_HandSolder -> footprints:C_0805_2012Metric_Pad1.18x1.45mm_HandSolder
- D1, D5, U$10, U$16, U$22, U$23, U$24: footprint Diode_SMD:D_SOD-123 -> footprints:D_SOD-123
- JP1, JP2, JP3, JP4: footprint Jumper:SolderJumper-2_P1.3mm_Open_TrianglePad1.0x1.5mm -> footprints:SolderJumper-2_P1.3mm_Open_TrianglePad1.0x1.5mm
- LED1, LED2, LED3, LED4, LED5, LED6, LED7: footprint Diode_SMD:D_0603_1608Metric_Pad1.05x0.95mm_HandSolder -> footprints:D_0603_1608Metric_Pad1.05x0.95mm_HandSolder
- R1, R10, R11, R12, R13, R14, R15, R16, R17, R18, R19, R2, R20, R22, R23, R25, R26, R27, R28, R30, R31, R36, R37, R5, R51, R54, R55, R56, R58, R6, R7, R8, R9: footprint Resistor_SMD:R_0603_1608Metric_Pad0.98x0.95mm_HandSolder -> footprints:R_0603_1608Metric_Pad0.98x0.95mm_HandSolder
- R21, R3, R4: footprint Resistor_SMD:R_2512_6332Metric_Pad1.40x3.35mm_HandSolder -> footprints:R_2512_6332Metric_Pad1.40x3.35mm_HandSolder
- TP1, TP13, TP14, TP15, TP2, TP3, TP4: footprint Connector_Pin:Pin_D1.3mm_L11.3mm_W2.8mm_Flat -> UNIVERSAL_JOINT:61-2348-11_0030
- TP10, TP11, TP12, TP16, TP17, TP5, TP6, TP7, TP8, TP9: footprint Connector_Pin:Pin_D1.2mm_L11.3mm_W3.0mm_Flat -> UNIVERSAL_JOINT:61-2348-11_0030
Connections:
- net at C1.1: now also U1.4 (CPH)
- net at C1.2: now also U1.3 (CPL)
Other:
- moved on the sheet: C1

Commit message: update to newest
Connections:
- net +3V3: now also C25.2, U2.3 (VCC)

Commit message: udpate
Parts:
- added U5: STM32G431CBU6, UNIVERSAL_JOINT:QFN50P700X700X65-49N-D, symbol STM32G431CBU6:STM32G431CBU6
Connections:
- net BRAKE: now also U5.12 (PA4); no longer U3.12 (PA4)
- net CS1: now also U5.19 (PB2); no longer U3.18 (PB2)
- net CURR_FB_U: now also U5.9 (PA1); no longer U3.9 (PA1)
- net CURR_FB_V: now also U5.24 (PB11); no longer U3.25 (PB11)
- net CURR_FB_W: now also U5.14 (PA6); no longer U3.14 (PA6)
- net DIP1: now also U5.3 (PC14-OSC32_IN); no longer U3.3 (PC14)
- net DIP2: now also U5.2 (PC13); no longer U3.2 (PC13)
- net DIP3: now also U5.43 (PB5); no longer U3.42 (PB5)
- net DIP4: now also U5.42 (PB4); no longer U3.41 (PB4)
- net FDCAN_RX: now also U5.33 (PA11); no longer U3.33 (PA11)
- net FDCAN_TX: now also U5.34 (PA12); no longer U3.34 (PA12)
- net H1: now also U5.44 (PB6); no longer U3.43 (PB6)
- net H2: now also U5.45 (PB7); no longer U3.44 (PB7)
- net JTDI: now also U5.38 (PA15); no longer U3.39 (PA15)
- net PWM_1: now also U5.30 (PA8); no longer U3.30 (PA8)
- net PWM_1N: now also U5.15 (PA7); no longer U3.15 (PA7)
- net PWM_2: now also U5.31 (PA9); no longer U3.31 (PA9)
- net PWM_2N: now also U5.17 (PB0); no longer U3.16 (PB0)
- net PWM_3: now also U5.32 (PA10); no longer U3.32 (PA10)
- net PWM_3N: now also U5.18 (PB1); no longer U3.17 (PB1)
- net SEC_IN: now also U5.4 (PC15-OSC32_OUT); no longer U3.4 (PC15)
- net SEC_OUT: now also U5.47 (PB9); no longer U3.46 (PB9)
- net SPI_MISO: now also U5.27 (PB14); no longer U3.28 (PB14)
- net SPI_MOSI: now also U5.28 (PB15); no longer U3.29 (PB15)
- net SPI_SCK: now also U5.26 (PB13); no longer U3.27 (PB13)
- net SWCLK/JTCK: now also U5.37 (PA14); no longer U3.38 (PA14)
- net SWDIO/JTMS: now also U5.36 (PA13); no longer U3.37 (PA13)
- net SWO/JTDO: now also U5.41 (PB3); no longer U3.40 (PB3)
- net TEMP: now also U5.13 (PA5); no longer U3.13 (PA5)
- net UART_RX: now also U5.11 (PA3); no longer U3.11 (PA3)
- net UART_TX: now also U5.10 (PA2); no longer U3.10 (PA2)
- net VBUS: now also U5.8 (PA0); no longer U3.8 (PA0)
- net at C23.2, X1.1: now also U5.5 (PF0-OSC_IN); no longer U3.5 (PF0-OSC_IN)
- net at C22.2, X1.3: now also U5.6 (PF1-OSC_OUT); no longer U3.6 (PF1-OSC_OUT)
- net at R20.2: now also U5.46 (PB8-BOOT0); no longer U3.45 (PB8-BOOT0)
- net at C24.2, R19.1, SW1.1 (1.1)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: now also U5.7 (PG10-NRST); no longer U3.7 (PG10-NRST)
Other:
- moved on the sheet: C22, C23, C24, R19, R20, SW1, U$16, X1
