File: UNIVERSAL_JOINT_v3_2/UNIVERSAL_JOINT_v3_2.kicad_pcb (KiCad board)
At the start: 4 copper layers, 76 x 75.9 mm, 158 parts, among them J1 M207810645, J12 FTSH-107-01-L-DV-K-TR, Q1 IAUC120N06S5L, Q2 IAUC120N06S5L, Q201 BSS138, Q202 BSS138, Q3 IAUC120N06S5L, Q4 IAUC120N06S5L, Q5 IAUC120N06S5L, Q6 IAUC120N06S5L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

Commit message: udpate
Parts:
- J1: value M207810645 -> M20-7810645
- U1: value QFN_IN32G4_STM -> STSPIN32G4
- U6: footprint Package_DFN_QFN:HVQFN-16-1EP_3x3mm_P0.5mm_EP1.5x1.5mm -> UNIVERSAL_JOINT:MA730GQ-Z
- X1: footprint Crystal:Crystal_SMD_2520-4Pin_2.5x2.0mm -> UNIVERSAL_JOINT:ECX-2236B2
