File: UNIVERSAL_JOINT_v3_2/UNIVERSAL_JOINT_v3_2.kicad_sch (KiCad schematic)
At the start: 158 parts, among them J1 M20-7810645, J12 FTSH-107-01-L-DV-K-TR, Q1 IAUC120N06S5L, Q2 IAUC120N06S5L, Q201 BSS138, Q202 BSS138, Q3 IAUC120N06S5L, Q4 IAUC120N06S5L, Q5 IAUC120N06S5L, Q6 IAUC120N06S5L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

Commit message: update descriptions
Other:
- note removed: "DODAĆ FILTR RC DO AB"
- note removed: "PRZY SCREF DODAĆ DZIELNIK - BRAK!"
- moved on the sheet: C19, C202, D205, D8, R211, R37, R39, TP14, TP15, TP16, TP17, TP3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

Commit message: udpate
Parts:
- U6: footprint Package_DFN_QFN:HVQFN-16-1EP_3x3mm_P0.5mm_EP1.5x1.5mm -> UNIVERSAL_JOINT:MA730GQ-Z
- X1: footprint Crystal:Crystal_SMD_2520-4Pin_2.5x2.0mm -> UNIVERSAL_JOINT:ECX-2236B2
Other:
- note removed: "NM"
Changed lines of the file:
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@@
     (stroke (width 0) (type default) (color 0 0 0 0))
   )
-  (wire (pts (xy 784.86 208.28) (xy 788.67 208.28))
-    (stroke (width 0) (type default) (color 0 0 0 0))
-  )
   (wire (pts (xy 783.59 24.13) (xy 783.59 26.67))
     (stroke (width 0) (type default) (color 0 0 0 0))
@@
     (stroke (width 0) (type default) (color 0 0 0 0))
   )
-  (wire (pts (xy 796.29 208.28) (xy 798.83 208.28))
-    (stroke (width 0) (type default) (color 0 0 0 0))
-  )
   (wire (pts (xy 885.19 343.535) (xy 885.19 346.075))
     (stroke (width 0) (type default) (color 0 0 0 0))
@@
     (stroke (width 0) (type default) (color 0 0 0 0))
   )
-  (wire (pts (xy 784.86 185.42) (xy 784.86 208.28))
-    (stroke (width 0) (type default) (color 0 0 0 0))
-  )
   (wire (pts (xy 774.7 245.745) (xy 774.7 250.19))
     (stroke (width 0) (type default) (color 0 0 0 0))
@@
     (effects (font (size 3 3)) (justify left bottom))
   )
-  (text "NM" (at 790.575 208.915 0)
-    (effects (font (size 1.27 1.27) (thickness 0.254) bold) (justify left bottom))
-  )
   (text "CONNECTORS" (at 49.53 163.83 0)
     (effects (font (size 3 3)) (justify left bottom))
@@
     (effects (font (size 1.27 1.27)) (justify left bottom))
   )
-  (text "NM" (at 775.335 174.625 0)
-    (effects (font (size 1.27 1.27) (thickness 0.254) bold) (justify left bottom))
-  )
   (text "A,B DODAĆ RC FILTER\n1k 10pF" (at 235.585 410.21 0)
     (effects (font (size 1.27 1.27)) (justify left bottom))
@@
   (symbol (lib_id "Connector:TestPoint_Probe") (at 494.03 317.5 0) (unit 1)
     (in_bom yes) (on_board yes)
-    (property "Reference" "TP24" (id 0) (at 498.475 314.6424 0)
+    (property "Reference" "TP24" (id 0) (at 496.57 316.865 0)
       (effects (font (size 1.27 1.27)) (justify left))
     )
-    (property "Value" "TestPoint_Probe" (id 1) (at 502.92 313.055 0)
+    (property "Value" "TestPoint_Probe" (id 1) (at 497.84 308.61 90)
       (effects (font (size 1.27 1.27)) (justify left))
     )
@@
       (effects (font (size 1.778 1.5113)) (justify right top))
     )
-    (property "Value" "1uF" (id 1) (at 505.714 309.499 0)
+    (property "Value" "1uF" (id 1) (at 506.73 310.515 0)
       (effects (font (size 1.778 1.5113)) (justify right top))
     )
@@
   (symbol (lib_id "Connector:TestPoint_Probe") (at 494.03 314.96 0) (unit 1)
     (in_bom yes) (on_board yes)
-    (property "Reference" "TP23" (id 0) (at 498.475 312.1024 0)
+    (property "Reference" "TP23" (id 0) (at 496.57 310.515 0)
       (effects (font (size 1.27 1.27)) (justify left))
     )
-    (property "Value" "TestPoint_Probe" (id 1) (at 502.92 310.515 0)
+    (property "Value" "TestPoint_Probe" (id 1) (at 497.84 308.61 90)
       (effects (font (size 1.27 1.27)) (justify left))
     )
@@
     (property "Reference" "U6" (id 0) (at 485.14 307.5644 0))
     (property "Value" "MA730" (id 1) (at 474.98 307.7995 0))
-    (property "Footprint" "Package_DFN_QFN:HVQFN-16-1EP_3x3mm_P0.5mm_EP1.5x1.5mm" (id 2) (at 481.33 344.17 0)
+    (property "Footprint" "UNIVERSAL_JOINT:MA730GQ-Z" (id 2) (at 481.33 344.17 0)
       (effects (font (size 1.27 1.27)) hide)
     )
@@
       (effects (font (size 1.27 1.27)) (justify left))
     )
-    (property "Footprint" "Crystal:Crystal_SMD_2520-4Pin_2.5x2.0mm" (id 2) (at 304.8 124.46 0)
+    (property "Footprint" "UNIVERSAL_JOINT:ECX-2236B2" (id 2) (at 304.8 124.46 0)
       (effects (font (size 1.27 1.27)) hide)
     )
@@
     )
     (path "/902147e1-3fee-47cd-9259-efa0e8ee0de0"
-      (reference "U6") (unit 1) (value "MA730") (footprint "Package_DFN_QFN:HVQFN-16-1EP_3x3mm_P0.5mm_EP1.5x1.5mm")
+      (reference "U6") (unit 1) (value "MA730") (footprint "UNIVERSAL_JOINT:MA730GQ-Z")
     )
     (path "/9124cc41-d0bb-4ac4-9425-1f1324ea8733"
-      (reference "X1") (unit 1) (value "ECS-240-8-36B2-CKM-TR") (footprint "Crystal:Crystal_SMD_2520-4Pin_2.5x2.0mm")
+      (reference "X1") (unit 1) (value "ECS-240-8-36B2-CKM-TR") (footprint "UNIVERSAL_JOINT:ECX-2236B2")
     )
   )
