File: UNIVERSAL_JOINT_v3_4/UNIVERSAL_JOINT_v3_4.kicad_pcb (KiCad board)
At the start: 4 copper layers, 76 x 75.9 mm, 180 parts, among them J1 BM02B-SRSS-TB, J12 FTSH-107-01-L-DV-K-TR, J2 BM02B-SRSS-TB, J3 Conn_01x11_Male, Q1 STL100N10, Q2 STL100N10, Q203 BSS138PS, Q3 STL100N10, Q4 STL100N10, Q5 STL100N10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

Commit message: UJ 3.5 - draft
Parts:
- U1: value STSPIN32G4 -> QFN_IN32G4_STM
