File: UNIVERSAL_JOINT_v3_5/UNIVERSAL_JOINT_v3_5.kicad_pcb (KiCad board)
At the start: 4 copper layers, 76 x 75.9 mm, 180 parts, among them J1 BM02B-SRSS-TB, J12 FTSH-107-01-L-DV-K-TR, J2 BM02B-SRSS-TB, J3 Conn_01x11_Male, Q1 STL100N10, Q2 STL100N10, Q203 BSS138PS, Q3 STL100N10, Q4 STL100N10, Q5 STL100N10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

Commit message: UJ 3.5 - draft
Parts:
- removed C25, C26, C27: 82nF 5%, footprints:C_0603_1608Metric_Pad1.08x0.95mm_HandSolder
- removed C34, C35: NM, footprints:C_0603_1608Metric_Pad1.08x0.95mm_HandSolder
- removed D10, D11, D9: BAT30K, footprints:D_0603_1608Metric_Pad1.05x0.95mm_HandSolder
- removed D12, D13: NM, footprints:D_0603_1608Metric_Pad1.05x0.95mm_HandSolder
- removed J12: FTSH-107-01-L-DV-K-TR, UNIVERSAL_JOINT:SAMTEC_FTSH-107-01-L-DV-K-TR
- removed R56, R58, R60: 68k 1%, footprints:R_0402_1005Metric_Pad0.72x0.64mm_HandSolder
- removed R57, R59, R61: 27k 1%, footprints:R_0402_1005Metric_Pad0.72x0.64mm_HandSolder
- removed R62, R63, R64: 3.9k 1%, footprints:R_0402_1005Metric_Pad0.72x0.64mm_HandSolder
- removed R81, R82: NM, footprints:R_0402_1005Metric_Pad0.72x0.64mm_HandSolder
- added J4: Conn_01x11_Male, footprints:PinHeader_1x09_P1.27mm_Vertical, F.Cu at (170.3, 94.8)
- added TC1: TC2030-IDC, UNIVERSAL_JOINT:TC2030-IDC, F.Cu at (126.6, 128.3)
- C202: footprint footprints:CP_Radial_D6.3mm_P2.50mm -> footprints:CP_Radial_D8.0mm_P2.50mm
- C217, C218: value C -> 100n
- J3: footprint footprints:PinHeader_1x11_P1.27mm_Vertical -> footprints:PinHeader_1x09_P1.27mm_Vertical
- R201, R202, R211, R212: footprint footprints:R_0402_1005Metric_Pad0.72x0.64mm_HandSolder -> footprints:R_0603_1608Metric_Pad0.98x0.95mm_HandSolder
- R37: value 72.3k 1% -> 92k 1%
- R39: value 3.01k 1% -> 3.9k 1%
- U1: value STSPIN32G4 -> QFN_IN32G4_STM
- moved SW3 22.2 mm to (120.4, 125.1), turned to -90 degrees
- moved J3 15.9 mm to (170.3, 115.2)
- moved R225 12.3 mm to (162.5, 125.7), turned to 180 degrees
- moved R226 11.5 mm to (164.9, 125.7), turned to 0 degrees
- moved L2 11.2 mm to (163.9, 123.7)
- moved U7 11.1 mm to (164.3, 120.4)
- moved C213 11.1 mm to (161.9, 123.5)
- moved C214 11.1 mm to (167.1, 120.6)
- moved D207 11.0 mm to (168.6, 120.6)
- moved C212 11.0 mm to (168.2, 123.4)
- moved R222 10.9 mm to (160.8, 120.4)
- moved R221 10.9 mm to (161.8, 120.4)
- moved C40 8.07 mm to (132.2, 130.6)
- moved D205 6.45 mm to (183.4, 108.4)
- moved R224 6.45 mm to (179.6, 107.1)
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Connections:
- J1 pad 1: +3V3 -> /MOTOR_TEMP
- J1 pad 2: /MOTOR_TEMP -> +3V3
- J3 pad 1: GND -> unconnected-(J3-Pad1)
- J3 pad 2: +5V -> unconnected-(J3-Pad2)
- J3 pad 3: +3V3 -> unconnected-(J3-Pad3)
- J3 pad 4: /SPI_SCK -> unconnected-(J3-Pad4)
- J3 pad 5: /SPI_MOSI -> unconnected-(J3-Pad5)
- J3 pad 6: /SPI_MISO -> unconnected-(J3-Pad6)
- J3 pad 7: /PC13 -> unconnected-(J3-Pad7)
- J3 pad 8: /PB9 -> /VCC
- J3 pad 9: /PB10 -> GND
- U1 pad 10: /VOUT2 -> unconnected-(U1-Pad10)
- U1 pad 11: /VOUT3 -> unconnected-(U1-Pad11)
- U1 pad 51: /JTDI -> /PA15
- U1 pad 57: /A_RC -> /A
- U1 pad 58: /B_RC -> /B
- U1 pad 9: /VOUT1 -> unconnected-(U1-Pad9)
Routing:
- net Net-(R56-Pad2): track 55.0 -> 0.00 mm, vias 2 -> 0
- net unconnected-(U1-Pad9): track 0.00 -> 52.7 mm, vias 0 -> 1
- net unconnected-(U1-Pad11): track 0.00 -> 49.7 mm, vias 0 -> 1
- net unconnected-(U1-Pad10): track 0.00 -> 49.0 mm, vias 0 -> 1
- net Net-(R58-Pad2): track 45.7 -> 0.00 mm, vias 2 -> 0
- net /A_RC: track 45.0 -> 0.00 mm, vias 2 -> 0
- net /PA15: track 0.00 -> 44.5 mm, vias 0 -> 1
- net /A: track 5.35 -> 47.6 mm, vias 1 -> 3
- net Net-(R60-Pad2): track 39.0 -> 0.00 mm, vias 2 -> 0
- net /B: track 5.25 -> 43.9 mm, vias 1 -> 3
- net /B_RC: track 38.4 -> 0.00 mm, vias 2 -> 0
- net /UART_TX: track 22.8 -> 54.0 mm, vias 2 -> 1
- net /UART_RX: track 23.7 -> 50.6 mm, vias 2 -> 1
- net /PA8: track 70.1 -> 44.9 mm, vias 2 -> 1
- net /PD2: track 64.0 -> 39.2 mm, vias 2 -> 1
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Other:
- outline, holes or cut-outs redrawn
- board text added: "+ dodatkowe SPI dla EtherCATa + rezystory przy ledach - 0603 + wydluzyc pady sensorow optycznych + rozsunac otoczenie sensorow optycznych - wymienic przycisk resetu + gniazdo programatora + uart na oddzielnych pinach"
- board text added: "v3.5"
- board text removed: "- dodatkowe SPI dla EtherCATa - EEPROM ?? dodac dodatkowy ?? - rezystory przy ledach - 0805 - wydluzyc pady sensorow optycznych - rozsunac otoczenie sensorow optycznych - wymienic przycisk resetu - gniazdo programatora - uart na oddzielnych pinach - gniazdo dodatkowego SPI dopasowac do SOM"
- board text removed: "v3.4"
