File: UNIVERSAL_JOINT_v3_5/UNIVERSAL_JOINT_v3_5.kicad_sch (KiCad schematic)
At the start: 180 parts, among them J1 BM02B-SRSS-TB, J12 FTSH-107-01-L-DV-K-TR, J2 BM02B-SRSS-TB, J3 Conn_01x11_Male, Q1 STL100N10, Q2 STL100N10, Q203 BSS138PS, Q3 STL100N10, Q4 STL100N10, Q5 STL100N10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

Commit message: UJ 3.5 - draft
Parts:
- removed C25, C26, C27: 82nF 5%, footprints:C_0603_1608Metric_Pad1.08x0.95mm_HandSolder, symbol Device:C
- removed C34, C35: NM, footprints:C_0603_1608Metric_Pad1.08x0.95mm_HandSolder, symbol Device:C
- removed D10, D11, D9: BAT30K, footprints:D_0603_1608Metric_Pad1.05x0.95mm_HandSolder, symbol Device:D_Schottky
- removed D12, D13: NM, footprints:D_0603_1608Metric_Pad1.05x0.95mm_HandSolder, symbol Device:D_Schottky
- removed J12: FTSH-107-01-L-DV-K-TR, UNIVERSAL_JOINT:SAMTEC_FTSH-107-01-L-DV-K-TR, symbol FTSH-107-01-L-DV-K-TR:FTSH-107-01-L-DV-K-TR
- removed R56, R58, R60: 68k 1%, footprints:R_0402_1005Metric_Pad0.72x0.64mm_HandSolder, symbol Device:R
- removed R57, R59, R61: 27k 1%, footprints:R_0402_1005Metric_Pad0.72x0.64mm_HandSolder, symbol Device:R
- removed R62, R63, R64: 3.9k 1%, footprints:R_0402_1005Metric_Pad0.72x0.64mm_HandSolder, symbol Device:R
- removed R81, R82: 0, footprints:R_0402_1005Metric_Pad0.72x0.64mm_HandSolder, symbol Device:R
- added J4: Conn_01x11_Male, footprints:PinHeader_1x09_P1.27mm_Vertical, symbol Connector:Conn_01x09_Male
- added TC1: TC2030-IDC, UNIVERSAL_JOINT:TC2030-IDC, symbol TC2030-IDC:TC2030-IDC
- C202: footprint footprints:CP_Radial_D6.3mm_P2.50mm -> footprints:CP_Radial_D8.0mm_P2.50mm
- J3: footprint footprints:PinHeader_1x11_P1.27mm_Vertical -> footprints:PinHeader_1x09_P1.27mm_Vertical; symbol Connector:Conn_01x11_Male -> Connector:Conn_01x09_Male
- Q1, Q2, Q3, Q4, Q5, Q6: footprint Package_TO_SOT_SMD:TDSON-8-1 -> footprints:TDSON-8-1
- R201, R202, R211, R212: footprint footprints:R_0402_1005Metric_Pad0.72x0.64mm_HandSolder -> footprints:R_0603_1608Metric_Pad0.98x0.95mm_HandSolder
Connections:
- net A_RC is gone; now on net A: U1.57 (PB6)
- net B_RC is gone; now on net B: U1.58 (PB7)
- net +3V3: now also J1.2, J4.8 (Pin_8); no longer J1.1, J3.3 (Pin_3)
- net +5V: now also J4.7 (Pin_7); no longer J3.2 (Pin_2)
- net GND: now also J3.9 (Pin_9), J4.9 (Pin_9), TC1.5 (GND); no longer J3.1 (Pin_1)
- net MOTOR_TEMP: now also J1.1; no longer J1.2
- net PA8: no longer J3.10 (Pin_10)
- net PB10: no longer J3.9 (Pin_9)
- net PB9: no longer J3.8 (Pin_8)
- net PC13: no longer J3.7 (Pin_7)
- net PD2: no longer J3.11 (Pin_11)
- net SPI_MISO: now also J4.3 (Pin_3); no longer J3.6 (Pin_6)
- net SPI_MOSI: now also J4.2 (Pin_2); no longer J3.5 (Pin_5)
- net SPI_SCK: now also J4.1 (Pin_1); no longer J3.4 (Pin_4)
- net SWCLK/JTCK: now also TC1.4 (SWCLK)
- net SWDIO/JTMS: now also TC1.2 (SWDIO)
- net SWO/JTDO: now also TC1.6 (SWO)
- net VCC: now also J3.8 (Pin_8)
- net nRST: now also TC1.3 (NRESET)
- net JTDI renamed PA15
- net VOUT1: no longer names the net of U1.9 (PC0)
- net VOUT2: no longer names the net of U1.10 (PC1)
- net VOUT3: no longer names the net of U1.11 (PC2)
Other:
- note removed: "A,B DODAĆ RC FILTER 1k 10pF"
